File: acsi_to_scsi/acsi_to_scsi.sch (KiCad schematic (older format))
At the start: 12 parts, among them J1 Conn_02x25_Odd_Even, U1 74ALS573, U10 74LS02, U11 74ALS74, U2 74ALS540, U3 74ALS540, U4 74LS01, U5 74ALS74, U6 74ALS08, U7 74ALS85, U8 74LS04, U9 74LS08

Commit message: a
Parts:
- added J?: Conn_01x19, symbol Connector_Generic:Conn_01x19
- added SW?: SW_DIP_x03, symbol Switch:SW_DIP_x03
Connections:
- net at U7.12 (A1): now also SW?.3
- net at U7.13 (A2): now also SW?.2
- net at U7.15 (A3): now also SW?.1
Other:
- moved on the sheet: J1, U10A, U10B, U10C, U10D, U10E, U11A, U11B, U11C, U4A, U4B, U4C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
