File: external_floppy/atari_floppy.kicad_pcb (KiCad board)
At the start: 2 copper layers, 7 parts, among them J1 12VDC, J3 DATA_IN, J4 FLOPPY, U1 L7805

Commit message: a
Parts:
- added J2: FLOPPY_PWR, atari_floppy:171826-4, F.Cu at (125.7, 109.2)
Connections:
- J1 pad 3: GND -> (no net)
Changed lines of the file:
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@@
     (tracks 19)
     (zones 0)
-    (modules 7)
+    (modules 8)
     (nets 25)
   )
@@
     (add_net "Net-(J4-Pad4)")
     (add_net "Net-(J4-Pad6)")
+  )
+  (module atari_floppy:171826-4 (layer F.Cu)
+    (at 125.73 109.22)
+    (descr "JST XH series connector, S4B-XH-A (http://www.jst-mfg.com/product/pdf/eng/eXH.pdf), generated with kicad-footprint-generator")
+    (tags "connector JST XH horizontal")
+    (fp_text reference J2 (at 6.25 -1.1) (layer F.SilkS)
+      (effects (font (size 1 1) (thickness 0.15)))
+    )
+    (fp_text value FLOPPY_PWR (at 5.2 14.4) (layer F.Fab)
+      (effects (font (size 1 1) (thickness 0.15)))
+    )
+    (fp_text user %R (at 4.85 6.35) (layer F.Fab)
+      (effects (font (size 1 1) (thickness 0.15)))
+    )
+    (fp_line (start 10 13.5) (end 10 0) (layer Dwgs.User) (width 0.12))
+    (fp_line (start 0 13.5) (end 10 13.5) (layer Dwgs.User) (width 0.12))
+    (fp_line (start 0 0) (end 0 13.5) (layer Dwgs.User) (width 0.12))
+    (fp_line (start 0 0) (end 10 0) (layer Dwgs.User) (width 0.12))
+    (fp_line (start -0.1 -0.1) (end 10.1 -0.1) (layer F.SilkS) (width 0.12))
+    (fp_line (start 10.1 -0.1) (end 10.1 13.6) (layer F.SilkS) (width 0.12))
+    (fp_line (start 10.1 13.6) (end -0.1 13.6) (layer F.SilkS) (width 0.12))
+    (fp_line (start -0.1 13.6) (end -0.1 -0.1) (layer F.SilkS) (width 0.12))
+    (pad 4 thru_hole oval (at 8.8 2.2) (size 1.7 1.95) (drill 0.95) (layers *.Cu *.Mask)
+      (net 2 +12V))
+    (pad 3 thru_hole oval (at 6.3 2.2) (size 1.7 1.95) (drill 0.95) (layers *.Cu *.Mask)
+      (net 1 GND))
+    (pad 2 thru_hole oval (at 3.8 2.2) (size 1.7 1.95) (drill 0.95) (layers *.Cu *.Mask)
+      (net 1 GND))
+    (pad 1 thru_hole roundrect (at 1.3 2.2) (size 1.7 1.95) (drill 0.95) (layers *.Cu *.Mask) (roundrect_rratio 0.147)
+      (net 3 +5V))
   )
   (module Package_TO_SOT_THT:TO-220-3_Horizontal_TabDown (layer F.Cu)
@@
     (fp_line (start 0.8 4.5) (end 0.8 -3.75) (layer F.Fab) (width 0.1))
     (fp_line (start 0 -4.5) (end -13.7 -4.5) (layer F.Fab) (width 0.1))
-    (pad 3 thru_hole roundrect (at -3 4.7 270) (size 3.5 3.5) (drill oval 3 1) (layers *.Cu *.Mask) (roundrect_rratio 0.25)
-      (net 1 GND))
+    (pad 3 thru_hole roundrect (at -3 4.7 270) (size 3.5 3.5) (drill oval 3 1) (layers *.Cu *.Mask) (roundrect_rratio 0.25))
     (pad 2 thru_hole roundrect (at -6 0 270) (size 3 3.5) (drill oval 1 3) (layers *.Cu *.Mask) (roundrect_rratio 0.25)
       (net 1 GND))
@@
       (effects (font (size 1 1) (thickness 0.15)))
     )
-    (fp_text user K (at 0 -2.1 90) (layer F.SilkS)
-      (effects (font (size 1 1) (thickness 0.15)))
-    )
+    (fp_text user K (at 0 -2.1 90) (layer F.Fab)
+      (effects (font (size 1 1) (thickness 0.15)))
+    )
