File: external_floppy/atari_st.kicad_sch (KiCad schematic)
At the start: 1 part

Commit message: a
Parts:
- removed J?: ADAPTER, symbol Connector_Generic:Conn_01x14
- added J5: ADAPTER, Connector_PinHeader_2.54mm:PinHeader_2x07_P2.54mm_Horizontal, symbol Connector_Generic:Conn_01x14
- added J6: ATARI, parts:DIN14, symbol Connector_Generic:Conn_01x14
Connections:
- net FLOPPY_DISKCHANGE: now also J5.1 (Pin_1)
- net FLOPPY_INDEX: now also J5.2 (Pin_2), J6.4 (Pin_4)
- net FLOPPY_MOTOR_ON: now also J5.5 (Pin_5), J6.8 (Pin_8)
- net FLOPPY_READY: now also J5.14 (Pin_14)
- net FLOPPY_READ_DATA: now also J5.12 (Pin_12), J6.1 (Pin_1)
- net FLOPPY_SELECT_A: now also J5.3 (Pin_3), J6.5 (Pin_5)
- net FLOPPY_SELECT_B: now also J5.4 (Pin_4), J6.6 (Pin_6)
- net FLOPPY_SIDE_SELECT: now also J5.13 (Pin_13), J6.2 (Pin_2)
- net FLOPPY_STEP: now also J5.7 (Pin_7), J6.10 (Pin_10)
- net FLOPPY_STEP_DIRECTION: now also J5.6 (Pin_6), J6.9 (Pin_9)
- net FLOPPY_TRACK_00: now also J5.10 (Pin_10), J6.13 (Pin_13)
- net FLOPPY_WRITE_DATA: now also J5.8 (Pin_8), J6.11 (Pin_11)
- net FLOPPY_WRITE_GATE: now also J5.9 (Pin_9), J6.12 (Pin_12)
- net FLOPPY_WRITE_PROTECT: now also J5.11 (Pin_11), J6.14 (Pin_14)
- new net GND: J6.3 (Pin_3), J6.7 (Pin_7)
- no-connect marks 0 -> 2
Changed lines of the file:
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@@
 (kicad_sch (version 20201015) (generator eeschema)
   (paper "A4")
+  (junction (at 138.43 87.63) (diameter 0.9144) (color 0 0 0 0))
+  (no_connect (at 121.92 52.07))
+  (no_connect (at 121.92 85.09))
   (wire (pts (xy 92.71 52.07) (xy 121.92 52.07))
     (stroke (width 0) (type solid) (color 0 0 0 0))
   )
-  (wire (pts (xy 92.71 54.61) (xy 121.92 54.61))
+  (wire (pts (xy 92.71 54.61) (xy 140.97 54.61))
     (stroke (width 0) (type solid) (color 0 0 0 0))
   )
-  (wire (pts (xy 92.71 57.15) (xy 121.92 57.15))
+  (wire (pts (xy 92.71 57.15) (xy 143.51 57.15))
     (stroke (width 0) (type solid) (color 0 0 0 0))
   )
-  (wire (pts (xy 92.71 59.69) (xy 121.92 59.69))
+  (wire (pts (xy 92.71 59.69) (xy 146.05 59.69))
     (stroke (width 0) (type solid) (color 0 0 0 0))
   )
-  (wire (pts (xy 92.71 69.85) (xy 121.92 69.85))
+  (wire (pts (xy 92.71 62.23) (xy 151.13 62.23))
     (stroke (width 0) (type solid) (color 0 0 0 0))
   )
-  (wire (pts (xy 92.71 74.93) (xy 121.92 74.93))
+  (wire (pts (xy 92.71 64.77) (xy 153.67 64.77))
     (stroke (width 0) (type solid) (color 0 0 0 0))
   )
-  (wire (pts (xy 92.71 80.01) (xy 121.92 80.01))
+  (wire (pts (xy 92.71 67.31) (xy 156.21 67.31))
     (stroke (width 0) (type solid) (color 0 0 0 0))
   )
-  (wire (pts (xy 121.92 62.23) (xy 92.71 62.23))
+  (wire (pts (xy 92.71 69.85) (xy 158.75 69.85))
     (stroke (width 0) (type solid) (color 0 0 0 0))
   )
-  (wire (pts (xy 121.92 64.77) (xy 92.71 64.77))
+  (wire (pts (xy 92.71 72.39) (xy 161.29 72.39))
     (stroke (width 0) (type solid) (color 0 0 0 0))
   )
-  (wire (pts (xy 121.92 67.31) (xy 92.71 67.31))
+  (wire (pts (xy 92.71 74.93) (xy 163.83 74.93))
     (stroke (width 0) (type solid) (color 0 0 0 0))
   )
-  (wire (pts (xy 121.92 72.39) (xy 92.71 72.39))
+  (wire (pts (xy 92.71 77.47) (xy 166.37 77.47))
     (stroke (width 0) (type solid) (color 0 0 0 0))
   )
-  (wire (pts (xy 121.92 77.47) (xy 92.71 77.47))
+  (wire (pts (xy 92.71 80.01) (xy 133.35 80.01))
     (stroke (width 0) (type solid) (color 0 0 0 0))
   )
-  (wire (pts (xy 121.92 82.55) (xy 92.71 82.55))
+  (wire (pts (xy 92.71 82.55) (xy 135.89 82.55))
     (stroke (width 0) (type solid) (color 0 0 0 0))
   )
   (wire (pts (xy 121.92 85.09) (xy 92.71 85.09))
+    (stroke (width 0) (type solid) (color 0 0 0 0))
+  )
+  (wire (pts (xy 127 87.63) (xy 127 95.25))
+    (stroke (width 0) (type solid) (color 0 0 0 0))
+  )
+  (wire (pts (xy 127 87.63) (xy 138.43 87.63))
+    (stroke (width 0) (type solid) (color 0 0 0 0))
+  )
+  (wire (pts (xy 133.35 90.17) (xy 133.35 80.01))
+    (stroke (width 0) (type solid) (color 0 0 0 0))
+  )
+  (wire (pts (xy 135.89 90.17) (xy 135.89 82.55))
+    (stroke (width 0) (type solid) (color 0 0 0 0))
+  )
+  (wire (pts (xy 138.43 87.63) (xy 138.43 90.17))
+    (stroke (width 0) (type solid) (color 0 0 0 0))
+  )
+  (wire (pts (xy 138.43 87.63) (xy 148.59 87.63))
+    (stroke (width 0) (type solid) (color 0 0 0 0))
+  )
+  (wire (pts (xy 140.97 90.17) (xy 140.97 54.61))
+    (stroke (width 0) (type solid) (color 0 0 0 0))
+  )
+  (wire (pts (xy 143.51 90.17) (xy 143.51 57.15))
+    (stroke (width 0) (type solid) (color 0 0 0 0))
+  )
+  (wire (pts (xy 146.05 90.17) (xy 146.05 59.69))
+    (stroke (width 0) (type solid) (color 0 0 0 0))
+  )
+  (wire (pts (xy 148.59 90.17) (xy 148.59 87.63))
+    (stroke (width 0) (type solid) (color 0 0 0 0))
+  )
+  (wire (pts (xy 151.13 90.17) (xy 151.13 62.23))
+    (stroke (width 0) (type solid) (color 0 0 0 0))
+  )
+  (wire (pts (xy 153.67 90.17) (xy 153.67 64.77))
+    (stroke (width 0) (type solid) (color 0 0 0 0))
+  )
+  (wire (pts (xy 156.21 90.17) (xy 156.21 67.31))
+    (stroke (width 0) (type solid) (color 0 0 0 0))
+  )
+  (wire (pts (xy 158.75 90.17) (xy 158.75 69.85))
+    (stroke (width 0) (type solid) (color 0 0 0 0))
+  )
+  (wire (pts (xy 161.29 90.17) (xy 161.29 72.39))
+    (stroke (width 0) (type solid) (color 0 0 0 0))
+  )
+  (wire (pts (xy 163.83 90.17) (xy 163.83 74.93))
+    (stroke (width 0) (type solid) (color 0 0 0 0))
+  )
+  (wire (pts (xy 166.37 77.47) (xy 166.37 90.17))
     (stroke (width 0) (type solid) (color 0 0 0 0))
   )
@@
     (effects (font (size 1.27 1.27)) (justify right bottom))
   )
+  (symbol (lib_id "power:GND") (at 127 95.25 0) (unit 1)
+    (in_bom yes) (on_board yes)
+    (property "Reference" "#PWR0101" (id 0) (at 127 101.6 0)
+      (effects (font (size 1.27 1.27)) hide)
+    )
+    (property "Value" "GND" (id 1) (at 128.27 100.33 0))
+    (property "Footprint" "" (id 2) (at 127 95.25 0)
+      (effects (font (size 1.27 1.27)) hide)
+    )
+    (property "Datasheet" "" (id 3) (at 127 95.25 0)
+      (effects (font (size 1.27 1.27)) hide)
+    )
+  )
   (symbol (lib_id "Connector_Generic:Conn_01x14") (at 87.63 67.31 0) (mirror y) (unit 1)
     (in_bom yes) (on_board yes)
-    (property "Reference" "J?" (id 0) (at 82.1182 68.6816 90))
+    (property "Reference" "J5" (id 0) (at 82.1182 68.6816 90))
     (property "Value" "ADAPTER" (id 1) (at 84.4296 68.6816 90))
-    (property "Footprint" "" (id 2) (at 87.63 67.31 0)
+    (property "Footprint" "Connector_PinHeader_2.54mm:PinHeader_2x07_P2.54mm_Horizontal" (id 2) (at 87.63 67.31 0)
       (effects (font (size 1.27 1.27)) hide)
     )
@@
       (effects (font (size 1.27 1.27)) hide)
     )
+  )
+  (symbol (lib_id "Connector_Generic:Conn_01x14") (at 148.59 95.25 90) (mirror x) (unit 1)
+    (in_bom yes) (on_board yes)
+    (property "Reference" "J6" (id 0) (at 149.86 97.79 0)
+      (effects (font (size 1.27 1.27)) (justify left))
+    )
+    (property "Value" "ATARI" (id 1) (at 152.4 97.79 0)
+      (effects (font (size 1.27 1.27)) (justify left))
+    )
+    (property "Footprint" "parts:DIN14" (id 2) (at 148.59 95.25 0)
+      (effects (font (size 1.27 1.27)) hide)
+    )
+    (property "Datasheet" "~" (id 3) (at 148.59 95.25 0)
+      (effects (font (size 1.27 1.27)) hide)
+    )
