File: external_floppy/atari_st.kicad_sch (KiCad schematic)
At the start: 2 parts, among them J5 ADAPTER, J6 ATARI

Commit message: a
Parts:
- removed J5: ADAPTER, Connector_PinHeader_2.54mm:PinHeader_2x07_P2.54mm_Horizontal, symbol Connector_Generic:Conn_01x14
- added J5: ADAPTER, Connector_IDC:IDC-Header_2x08_P2.54mm_Vertical, symbol Connector_Generic:Conn_01x16
Connections:
- net FLOPPY_DISKCHANGE: now also J5.1 (Pin_1)
- net FLOPPY_INDEX: now also J5.2 (Pin_2)
- net FLOPPY_MOTOR_ON: now also J5.5 (Pin_5)
- net FLOPPY_READY: now also J5.14 (Pin_14)
- net FLOPPY_READ_DATA: now also J5.12 (Pin_12)
- net FLOPPY_SELECT_A: now also J5.3 (Pin_3)
- net FLOPPY_SELECT_B: now also J5.4 (Pin_4)
- net FLOPPY_SIDE_SELECT: now also J5.13 (Pin_13)
- net FLOPPY_STEP: now also J5.7 (Pin_7)
- net FLOPPY_STEP_DIRECTION: now also J5.6 (Pin_6)
- net FLOPPY_TRACK_00: now also J5.10 (Pin_10)
- net FLOPPY_WRITE_DATA: now also J5.8 (Pin_8)
- net FLOPPY_WRITE_GATE: now also J5.9 (Pin_9)
- net FLOPPY_WRITE_PROTECT: now also J5.11 (Pin_11)
- net GND: now also J5.16 (Pin_16)
- no-connect marks 2 -> 3
Changed lines of the file:
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@@
   (no_connect (at 121.92 52.07))
   (no_connect (at 121.92 85.09))
+  (no_connect (at 92.71 87.63))
   (wire (pts (xy 92.71 52.07) (xy 121.92 52.07))
     (stroke (width 0) (type solid) (color 0 0 0 0))
@@
   )
   (wire (pts (xy 92.71 82.55) (xy 135.89 82.55))
+    (stroke (width 0) (type solid) (color 0 0 0 0))
+  )
+  (wire (pts (xy 95.25 90.17) (xy 92.71 90.17))
+    (stroke (width 0) (type solid) (color 0 0 0 0))
+  )
+  (wire (pts (xy 95.25 95.25) (xy 95.25 90.17))
     (stroke (width 0) (type solid) (color 0 0 0 0))
   )
@@
     (effects (font (size 1.27 1.27)) (justify right bottom))
   )
+  (symbol (lib_id "power:GND") (at 95.25 95.25 0) (unit 1)
+    (in_bom yes) (on_board yes)
+    (property "Reference" "#PWR0103" (id 0) (at 95.25 101.6 0)
+      (effects (font (size 1.27 1.27)) hide)
+    )
+    (property "Value" "GND" (id 1) (at 96.52 100.33 0))
+    (property "Footprint" "" (id 2) (at 95.25 95.25 0)
+      (effects (font (size 1.27 1.27)) hide)
+    )
+    (property "Datasheet" "" (id 3) (at 95.25 95.25 0)
+      (effects (font (size 1.27 1.27)) hide)
+    )
+  )
   (symbol (lib_id "power:GND") (at 127 95.25 0) (unit 1)
     (in_bom yes) (on_board yes)
@@
     )
     (property "Datasheet" "" (id 3) (at 127 95.25 0)
-      (effects (font (size 1.27 1.27)) hide)
-    )
-  )
-  (symbol (lib_id "Connector_Generic:Conn_01x14") (at 87.63 67.31 0) (mirror y) (unit 1)
-    (in_bom yes) (on_board yes)
-    (property "Reference" "J5" (id 0) (at 82.1182 68.6816 90))
-    (property "Value" "ADAPTER" (id 1) (at 84.4296 68.6816 90))
-    (property "Footprint" "Connector_PinHeader_2.54mm:PinHeader_2x07_P2.54mm_Horizontal" (id 2) (at 87.63 67.31 0)
-      (effects (font (size 1.27 1.27)) hide)
-    )
-    (property "Datasheet" "~" (id 3) (at 87.63 67.31 0)
       (effects (font (size 1.27 1.27)) hide)
     )
@@
       (effects (font (size 1.27 1.27)) hide)
     )
+  )
+  (symbol (lib_id "Connector_Generic:Conn_01x16") (at 87.63 69.85 0) (mirror y) (unit 1)
+    (in_bom yes) (on_board yes)
+    (property "Reference" "J5" (id 0) (at 90.17 45.72 0))
+    (property "Value" "ADAPTER" (id 1) (at 90.17 48.26 0))
+    (property "Footprint" "Connector_IDC:IDC-Header_2x08_P2.54mm_Vertical" (id 2) (at 87.63 69.85 0)
+      (effects (font (size 1.27 1.27)) hide)
+    )
+    (property "Datasheet" "~" (id 3) (at 87.63 69.85 0)
+      (effects (font (size 1.27 1.27)) hide)
+    )
