File: external_floppy/floppy.kicad_sch (KiCad schematic)
At the start: 8 parts, among them J1 12VDC, J2 FLOPPY_PWR, J4 FLOPPY, U1 L7805

Commit message: a
Parts:
- added SW? (x2): SW_DPDT_x2, symbol Switch:SW_DPDT_x2
Connections:
- net FLOPPY_SELECT_A: now also SW?.1 (A), SW?.6 (C); no longer J4.10 (Pin_10)
- net FLOPPY_SELECT_B: now also SW?.3 (C), SW?.4 (A); no longer J4.12 (Pin_12)
- new net F_INSEL_A: J4.10 (Pin_10), SW?.2 (B)
- new net F_INSEL_B: J4.12 (Pin_12), SW?.5 (B)
Changed lines of the file:
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@@
   (junction (at 134.62 85.09) (diameter 0.9144) (color 0 0 0 0))
   (no_connect (at 121.92 59.69))
+  (no_connect (at 134.62 44.45))
+  (no_connect (at 121.92 49.53))
   (no_connect (at 121.92 46.99))
-  (no_connect (at 121.92 49.53))
-  (no_connect (at 134.62 44.45))
   (wire (pts (xy 26.67 63.5) (xy 26.67 60.96))
     (stroke (width 0) (type solid) (color 0 0 0 0))
@@
     (stroke (width 0) (type solid) (color 0 0 0 0))
   )
-  (wire (pts (xy 100.33 54.61) (xy 100.33 57.15))
-    (stroke (width 0) (type solid) (color 0 0 0 0))
-  )
-  (wire (pts (xy 100.33 57.15) (xy 92.71 57.15))
-    (stroke (width 0) (type solid) (color 0 0 0 0))
-  )
-  (wire (pts (xy 102.87 57.15) (xy 102.87 59.69))
-    (stroke (width 0) (type solid) (color 0 0 0 0))
-  )
-  (wire (pts (xy 102.87 59.69) (xy 92.71 59.69))
-    (stroke (width 0) (type solid) (color 0 0 0 0))
-  )
   (wire (pts (xy 121.92 44.45) (xy 95.25 44.45))
     (stroke (width 0) (type solid) (color 0 0 0 0))
@@
     (stroke (width 0) (type solid) (color 0 0 0 0))
   )
-  (wire (pts (xy 121.92 54.61) (xy 100.33 54.61))
-    (stroke (width 0) (type solid) (color 0 0 0 0))
-  )
-  (wire (pts (xy 121.92 57.15) (xy 102.87 57.15))
-    (stroke (width 0) (type solid) (color 0 0 0 0))
-  )
   (wire (pts (xy 121.92 62.23) (xy 92.71 62.23))
     (stroke (width 0) (type solid) (color 0 0 0 0))
@@
     (stroke (width 0) (type solid) (color 0 0 0 0))
   )
+  (label "F_INSEL_A" (at 64.77 100.33 180)
+    (effects (font (size 1.27 1.27)) (justify right bottom))
+  )
+  (label "F_INSEL_B" (at 64.77 114.3 180)
+    (effects (font (size 1.27 1.27)) (justify right bottom))
+  )
+  (label "FLOPPY_SELECT_A" (at 74.93 97.79 0)
+    (effects (font (size 1.27 1.27)) (justify left bottom))
+  )
+  (label "FLOPPY_SELECT_B" (at 74.93 102.87 0)
+    (effects (font (size 1.27 1.27)) (justify left bottom))
+  )
+  (label "FLOPPY_SELECT_B" (at 74.93 111.76 0)
+    (effects (font (size 1.27 1.27)) (justify left bottom))
+  )
+  (label "FLOPPY_SELECT_A" (at 74.93 116.84 0)
+    (effects (font (size 1.27 1.27)) (justify left bottom))
+  )
+  (label "FLOPPY_SELECT_A" (at 92.71 57.15 0)
+    (effects (font (size 1.27 1.27)) (justify left bottom))
+  )
+  (label "FLOPPY_SELECT_B" (at 92.71 59.69 0)
+    (effects (font (size 1.27 1.27)) (justify left bottom))
+  )
   (label "FLOPPY_DISKCHANGE" (at 121.92 44.45 180)
     (effects (font (size 1.27 1.27)) (justify right bottom))
@@
     (effects (font (size 1.27 1.27)) (justify right bottom))
   )
-  (label "FLOPPY_SELECT_A" (at 121.92 54.61 180)
-    (effects (font (size 1.27 1.27)) (justify right bottom))
-  )
-  (label "FLOPPY_SELECT_B" (at 121.92 57.15 180)
+  (label "F_INSEL_A" (at 121.92 54.61 180)
+    (effects (font (size 1.27 1.27)) (justify right bottom))
+  )
+  (label "F_INSEL_B" (at 121.92 57.15 180)
     (effects (font (size 1.27 1.27)) (justify right bottom))
   )
@@
     )
     (property "Datasheet" "~" (id 3) (at 29.21 68.58 0)
+      (effects (font (size 1.27 1.27)) hide)
+    )
+  )
+  (symbol (lib_id "Switch:SW_DPDT_x2") (at 69.85 100.33 0) (unit 1)
+    (in_bom yes) (on_board yes)
+    (property "Reference" "SW?" (id 0) (at 69.85 92.71 0))
+    (property "Value" "SW_DPDT_x2" (id 1) (at 69.85 95.25 0))
+    (property "Footprint" "" (id 2) (at 69.85 100.33 0)
+      (effects (font (size 1.27 1.27)) hide)
+    )
+    (property "Datasheet" "~" (id 3) (at 69.85 100.33 0)
+      (effects (font (size 1.27 1.27)) hide)
+    )
+  )
+  (symbol (lib_id "Switch:SW_DPDT_x2") (at 69.85 114.3 0) (unit 2)
+    (in_bom yes) (on_board yes)
+    (property "Reference" "SW?" (id 0) (at 69.85 106.68 0))
+    (property "Value" "SW_DPDT_x2" (id 1) (at 69.85 109.22 0))
+    (property "Footprint" "" (id 2) (at 69.85 114.3 0)
+      (effects (font (size 1.27 1.27)) hide)
+    )
+    (property "Datasheet" "~" (id 3) (at 69.85 114.3 0)
       (effects (font (size 1.27 1.27)) hide)
     )
@@
       (reference "J?") (unit 1) (value "ADAPTER") (footprint "")
     )
+    (path "/ebd9fdfc-3919-4a03-8180-54d97bd03282"
+      (reference "SW?") (unit 1) (value "SW_DPDT_x2") (footprint "")
+    )
+    (path "/60153e7c-7d60-42d1-a9fe-98c5063cb180"
+      (reference "SW?") (unit 2) (value "SW_DPDT_x2") (footprint "")
+    )
     (path "/00000000-0000-0000-0000-00005fc363e4"

Commit message: a
Parts:
- J3: renamed from J?; footprint (none) -> Connector_PinHeader_2.54mm:PinHeader_2x07_P2.54mm_Vertical
- gave numbers to parts that had none: 1
Changed lines of the file:
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@@
   (junction (at 134.62 85.09) (diameter 0.9144) (color 0 0 0 0))
   (no_connect (at 121.92 59.69))
+  (no_connect (at 121.92 46.99))
+  (no_connect (at 121.92 49.53))
   (no_connect (at 134.62 44.45))
-  (no_connect (at 121.92 49.53))
-  (no_connect (at 121.92 46.99))
   (wire (pts (xy 26.67 63.5) (xy 26.67 60.96))
     (stroke (width 0) (type solid) (color 0 0 0 0))
@@
   (symbol (lib_id "Switch:SW_DPDT_x2") (at 69.85 100.33 0) (unit 1)
     (in_bom yes) (on_board yes)
-    (property "Reference" "SW?" (id 0) (at 69.85 92.71 0))
+    (property "Reference" "SW1" (id 0) (at 69.85 92.71 0))
     (property "Value" "SW_DPDT_x2" (id 1) (at 69.85 95.25 0))
     (property "Footprint" "" (id 2) (at 69.85 100.33 0)
@@
   (symbol (lib_id "Switch:SW_DPDT_x2") (at 69.85 114.3 0) (unit 2)
     (in_bom yes) (on_board yes)
-    (property "Reference" "SW?" (id 0) (at 69.85 106.68 0))
+    (property "Reference" "SW1" (id 0) (at 69.85 106.68 0))
     (property "Value" "SW_DPDT_x2" (id 1) (at 69.85 109.22 0))
     (property "Footprint" "" (id 2) (at 69.85 114.3 0)
@@
   (symbol (lib_id "Connector_Generic:Conn_01x14") (at 87.63 67.31 0) (mirror y) (unit 1)
     (in_bom yes) (on_board yes)
-    (property "Reference" "J?" (id 0) (at 82.1182 68.6816 90))
+    (property "Reference" "J3" (id 0) (at 82.1182 68.6816 90))
     (property "Value" "ADAPTER" (id 1) (at 84.4296 68.6816 90))
-    (property "Footprint" "" (id 2) (at 87.63 67.31 0)
+    (property "Footprint" "Connector_PinHeader_2.54mm:PinHeader_2x07_P2.54mm_Vertical" (id 2) (at 87.63 67.31 0)
       (effects (font (size 1.27 1.27)) hide)
     )
@@
       (reference "J2") (unit 1) (value "FLOPPY_PWR") (footprint "atari_floppy:171826-4")
     )
+    (path "/00000000-0000-0000-0000-00005fe91e46"
+      (reference "J3") (unit 1) (value "ADAPTER") (footprint "Connector_PinHeader_2.54mm:PinHeader_2x07_P2.54mm_Vertical")
+    )
     (path "/00000000-0000-0000-0000-00005fc468f3"
       (reference "J4") (unit 1) (value "FLOPPY") (footprint "Connector_PinHeader_2.54mm:PinHeader_2x17_P2.54mm_Horizontal")
     )
-    (path "/00000000-0000-0000-0000-00005fe91e46"
-      (reference "J?") (unit 1) (value "ADAPTER") (footprint "")
-    )
     (path "/ebd9fdfc-3919-4a03-8180-54d97bd03282"
-      (reference "SW?") (unit 1) (value "SW_DPDT_x2") (footprint "")
+      (reference "SW1") (unit 1) (value "SW_DPDT_x2") (footprint "")
     )
     (path "/60153e7c-7d60-42d1-a9fe-98c5063cb180"
-      (reference "SW?") (unit 2) (value "SW_DPDT_x2") (footprint "")
+      (reference "SW1") (unit 2) (value "SW_DPDT_x2") (footprint "")
     )
     (path "/00000000-0000-0000-0000-00005fc363e4"
       (reference "U1") (unit 1) (value "L7805") (footprint "Package_TO_SOT_THT:TO-220-3_Horizontal_TabDown")
     )
-    (path "/214e5bd1-de3c-4ec2-8553-5b0be1a71a0f/00000000-0000-0000-0000-00005fe91e46"
-      (reference "J?") (unit 1) (value "ADAPTER") (footprint "")
-    )
-  )
+    (path "/214e5bd1-de3c-4ec2-8553-5b0be1a71a0f/278b2b95-eb2b-4c5f-bd49-6d46efcc2c1d"
+      (reference "#PWR0101") (unit 1) (value "GND") (footprint "")
+    )
+    (path "/214e5bd1-de3c-4ec2-8553-5b0be1a71a0f/0cefa351-cb06-47b9-89b0-293bb017abf7"
+      (reference "J5") (unit 1) (value "ADAPTER") (footprint "Connector_PinHeader_2.54mm:PinHeader_2x07_P2.54mm_Horizontal")
+    )
+    (path "/214e5bd1-de3c-4ec2-8553-5b0be1a71a0f/3e20fa31-0809-47c3-be37-022bd242ab1a"
+      (reference "J6") (unit 1) (value "ATARI") (footprint "parts:DIN14")
+    )
+  )

Commit message: a
Parts:
- removed J3: ADAPTER, Connector_PinHeader_2.54mm:PinHeader_2x07_P2.54mm_Vertical, symbol Connector_Generic:Conn_01x14
- added J3: ADAPTER, Connector_IDC:IDC-Header_2x08_P2.54mm_Horizontal, symbol Connector_Generic:Conn_01x16
Connections:
- net +5V: now also J3.15 (Pin_15)
- net FLOPPY_DISKCHANGE: now also J3.1 (Pin_1)
- net FLOPPY_INDEX: now also J3.2 (Pin_2)
- net FLOPPY_MOTOR_ON: now also J3.5 (Pin_5)
- net FLOPPY_READY: now also J3.14 (Pin_14)
- net FLOPPY_READ_DATA: now also J3.12 (Pin_12)
- net FLOPPY_SELECT_A: now also J3.3 (Pin_3)
- net FLOPPY_SELECT_B: now also J3.4 (Pin_4)
- net FLOPPY_SIDE_SELECT: now also J3.13 (Pin_13)
- net FLOPPY_STEP: now also J3.7 (Pin_7)
- net FLOPPY_STEP_DIRECTION: now also J3.6 (Pin_6)
- net FLOPPY_TRACK_00: now also J3.10 (Pin_10)
- net FLOPPY_WRITE_DATA: now also J3.8 (Pin_8)
- net FLOPPY_WRITE_GATE: now also J3.9 (Pin_9)
- net FLOPPY_WRITE_PROTECT: now also J3.11 (Pin_11)
- net GND: now also J3.16 (Pin_16)
Other:
- moved on the sheet: SW1A, SW1B
Changed lines of the file:
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@@
+    (stroke (width 0) (type solid) (color 0 0 0 0))
+  )
+  (wire (pts (xy 92.71 90.17) (xy 95.25 90.17))
     (stroke (width 0) (type solid) (color 0 0 0 0))
   )
@@
     (stroke (width 0) (type solid) (color 0 0 0 0))
   )
-  (label "F_INSEL_A" (at 64.77 100.33 180)
-    (effects (font (size 1.27 1.27)) (justify right bottom))
-  )
-  (label "F_INSEL_B" (at 64.77 114.3 180)
-    (effects (font (size 1.27 1.27)) (justify right bottom))
-  )
-  (label "FLOPPY_SELECT_A" (at 74.93 97.79 0)
-    (effects (font (size 1.27 1.27)) (justify left bottom))
-  )
-  (label "FLOPPY_SELECT_B" (at 74.93 102.87 0)
-    (effects (font (size 1.27 1.27)) (justify left bottom))
-  )
-  (label "FLOPPY_SELECT_B" (at 74.93 111.76 0)
-    (effects (font (size 1.27 1.27)) (justify left bottom))
-  )
-  (label "FLOPPY_SELECT_A" (at 74.93 116.84 0)
+  (label "F_INSEL_A" (at 36.83 113.03 180)
+    (effects (font (size 1.27 1.27)) (justify right bottom))
+  )
+  (label "F_INSEL_B" (at 36.83 127 180)
+    (effects (font (size 1.27 1.27)) (justify right bottom))
+  )
+  (label "FLOPPY_SELECT_A" (at 46.99 110.49 0)
+    (effects (font (size 1.27 1.27)) (justify left bottom))
+  )
+  (label "FLOPPY_SELECT_B" (at 46.99 115.57 0)
+    (effects (font (size 1.27 1.27)) (justify left bottom))
+  )
+  (label "FLOPPY_SELECT_B" (at 46.99 124.46 0)
+    (effects (font (size 1.27 1.27)) (justify left bottom))
+  )
+  (label "FLOPPY_SELECT_A" (at 46.99 129.54 0)
     (effects (font (size 1.27 1.27)) (justify left bottom))
   )
@@
   )
   (label "FLOPPY_SELECT_B" (at 92.71 59.69 0)
+    (effects (font (size 1.27 1.27)) (justify left bottom))
+  )
+  (label "+5V" (at 92.71 87.63 0)
     (effects (font (size 1.27 1.27)) (justify left bottom))
   )
@@
     )
     (property "Datasheet" "" (id 3) (at 62.23 43.18 0)
+      (effects (font (size 1.27 1.27)) hide)
+    )
+  )
+  (symbol (lib_id "power:GND") (at 95.25 90.17 0) (unit 1)
+    (in_bom yes) (on_board yes)
+    (property "Reference" "#PWR0102" (id 0) (at 95.25 96.52 0)
+      (effects (font (size 1.27 1.27)) hide)
+    )
+    (property "Value" "GND" (id 1) (at 96.52 95.25 0))
+    (property "Footprint" "" (id 2) (at 95.25 90.17 0)
+      (effects (font (size 1.27 1.27)) hide)
+    )
+    (property "Datasheet" "" (id 3) (at 95.25 90.17 0)
       (effects (font (size 1.27 1.27)) hide)
     )
@@
     )
   )
-  (symbol (lib_id "Switch:SW_DPDT_x2") (at 69.85 100.33 0) (unit 1)
-    (in_bom yes) (on_board yes)
-    (property "Reference" "SW1" (id 0) (at 69.85 92.71 0))
-    (property "Value" "SW_DPDT_x2" (id 1) (at 69.85 95.25 0))
-    (property "Footprint" "" (id 2) (at 69.85 100.33 0)
-      (effects (font (size 1.27 1.27)) hide)
-    )
-    (property "Datasheet" "~" (id 3) (at 69.85 100.33 0)
-      (effects (font (size 1.27 1.27)) hide)
-    )
-  )
-  (symbol (lib_id "Switch:SW_DPDT_x2") (at 69.85 114.3 0) (unit 2)
-    (in_bom yes) (on_board yes)
-    (property "Reference" "SW1" (id 0) (at 69.85 106.68 0))
-    (property "Value" "SW_DPDT_x2" (id 1) (at 69.85 109.22 0))
-    (property "Footprint" "" (id 2) (at 69.85 114.3 0)
-      (effects (font (size 1.27 1.27)) hide)
-    )
-    (property "Datasheet" "~" (id 3) (at 69.85 114.3 0)
+  (symbol (lib_id "Switch:SW_DPDT_x2") (at 41.91 113.03 0) (unit 1)
+    (in_bom yes) (on_board yes)
+    (property "Reference" "SW1" (id 0) (at 41.91 105.41 0))
+    (property "Value" "SW_DPDT_x2" (id 1) (at 41.91 107.95 0))
+    (property "Footprint" "" (id 2) (at 41.91 113.03 0)
+      (effects (font (size 1.27 1.27)) hide)
+    )
+    (property "Datasheet" "~" (id 3) (at 41.91 113.03 0)
+      (effects (font (size 1.27 1.27)) hide)
+    )
+  )
+  (symbol (lib_id "Switch:SW_DPDT_x2") (at 41.91 127 0) (unit 2)
+    (in_bom yes) (on_board yes)
+    (property "Reference" "SW1" (id 0) (at 41.91 119.38 0))
+    (property "Value" "SW_DPDT_x2" (id 1) (at 41.91 121.92 0))
+    (property "Footprint" "" (id 2) (at 41.91 127 0)
+      (effects (font (size 1.27 1.27)) hide)
+    )
+    (property "Datasheet" "~" (id 3) (at 41.91 127 0)
       (effects (font (size 1.27 1.27)) hide)
     )
@@
     )
   )
-  (symbol (lib_id "Connector_Generic:Conn_01x14") (at 87.63 67.31 0) (mirror y) (unit 1)
-    (in_bom yes) (on_board yes)
-    (property "Reference" "J3" (id 0) (at 82.1182 68.6816 90))
-    (property "Value" "ADAPTER" (id 1) (at 84.4296 68.6816 90))
-    (property "Footprint" "Connector_PinHeader_2.54mm:PinHeader_2x07_P2.54mm_Vertical" (id 2) (at 87.63 67.31 0)
-      (effects (font (size 1.27 1.27)) hide)
-    )
-    (property "Datasheet" "~" (id 3) (at 87.63 67.31 0)
+  (symbol (lib_id "Connector_Generic:Conn_01x16") (at 87.63 69.85 0) (mirror y) (unit 1)
+    (in_bom yes) (on_board yes)
+    (property "Reference" "J3" (id 0) (at 90.17 45.72 0))
+    (property "Value" "ADAPTER" (id 1) (at 90.17 48.26 0))
+    (property "Footprint" "Connector_IDC:IDC-Header_2x08_P2.54mm_Horizontal" (id 2) (at 87.63 69.85 0)
+      (effects (font (size 1.27 1.27)) hide)
+    )
+    (property "Datasheet" "~" (id 3) (at 87.63 69.85 0)
       (effects (font (size 1.27 1.27)) hide)
     )
@@
       (reference "#PWR07") (unit 1) (value "GND") (footprint "")
     )
+    (path "/ceeac992-fc29-4a73-9f03-f51f466531c4"
+      (reference "#PWR0102") (unit 1) (value "GND") (footprint "")
+    )
     (path "/00000000-0000-0000-0000-00005fc399bb"
       (reference "C1") (unit 1) (value "470uF") (footprint "Capacitor_THT:C_Radial_D10.0mm_H12.5mm_P5.00mm")
@@
       (reference "J2") (unit 1) (value "FLOPPY_PWR") (footprint "atari_floppy:171826-4")
     )
-    (path "/00000000-0000-0000-0000-00005fe91e46"
-      (reference "J3") (unit 1) (value "ADAPTER") (footprint "Connector_PinHeader_2.54mm:PinHeader_2x07_P2.54mm_Vertical")
+    (path "/afba136e-7f84-4ff1-b6f4-6a1445c64da2"
+      (reference "J3") (unit 1) (value "ADAPTER") (footprint "Connector_IDC:IDC-Header_2x08_P2.54mm_Horizontal")
     )
     (path "/00000000-0000-0000-0000-00005fc468f3"
@@
       (reference "#PWR0101") (unit 1) (value "GND") (footprint "")
     )
-    (path "/214e5bd1-de3c-4ec2-8553-5b0be1a71a0f/0cefa351-cb06-47b9-89b0-293bb017abf7"
-      (reference "J5") (unit 1) (value "ADAPTER") (footprint "Connector_PinHeader_2.54mm:PinHeader_2x07_P2.54mm_Horizontal")
+    (path "/214e5bd1-de3c-4ec2-8553-5b0be1a71a0f/507d2933-082b-4fad-ad51-d42819335b4a"
+      (reference "#PWR0103") (unit 1) (value "GND") (footprint "")
+    )
+    (path "/214e5bd1-de3c-4ec2-8553-5b0be1a71a0f/e4d3af14-b01c-4ff2-907e-cbfc6e32f0ec"
+      (reference "J5") (unit 1) (value "ADAPTER") (footprint "Connector_IDC:IDC-Header_2x08_P2.54mm_Vertical")
     )
     (path "/214e5bd1-de3c-4ec2-8553-5b0be1a71a0f/3e20fa31-0809-47c3-be37-022bd242ab1a"

Commit message: a
Parts:
- J4: footprint Connector_PinHeader_2.54mm:PinHeader_2x17_P2.54mm_Horizontal -> Connector_IDC:IDC-Header_2x17_P2.54mm_Vertical
- SW1: footprint (none) -> Button_Switch_THT:SW_CuK_JS202011AQN_DPDT_Angled
Changed lines of the file:
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@@
   (junction (at 134.62 82.55) (diameter 0.9144) (color 0 0 0 0))
   (junction (at 134.62 85.09) (diameter 0.9144) (color 0 0 0 0))
-  (no_connect (at 121.92 59.69))
   (no_connect (at 121.92 46.99))
   (no_connect (at 121.92 49.53))
   (no_connect (at 134.62 44.45))
+  (no_connect (at 121.92 59.69))
   (wire (pts (xy 26.67 63.5) (xy 26.67 60.96))
     (stroke (width 0) (type solid) (color 0 0 0 0))
@@
     (property "Reference" "SW1" (id 0) (at 41.91 105.41 0))
     (property "Value" "SW_DPDT_x2" (id 1) (at 41.91 107.95 0))
-    (property "Footprint" "" (id 2) (at 41.91 113.03 0)
+    (property "Footprint" "Button_Switch_THT:SW_CuK_JS202011AQN_DPDT_Angled" (id 2) (at 41.91 113.03 0)
       (effects (font (size 1.27 1.27)) hide)
     )
@@
     (property "Reference" "SW1" (id 0) (at 41.91 119.38 0))
     (property "Value" "SW_DPDT_x2" (id 1) (at 41.91 121.92 0))
-    (property "Footprint" "" (id 2) (at 41.91 127 0)
+    (property "Footprint" "Button_Switch_THT:SW_CuK_JS202011AQN_DPDT_Angled" (id 2) (at 41.91 127 0)
       (effects (font (size 1.27 1.27)) hide)
     )
@@
       (effects (font (size 1.27 1.27)) (justify left))
     )
-    (property "Footprint" "Connector_PinHeader_2.54mm:PinHeader_2x17_P2.54mm_Horizontal" (id 2) (at 129.54 64.77 0)
+    (property "Footprint" "Connector_IDC:IDC-Header_2x17_P2.54mm_Vertical" (id 2) (at 129.54 64.77 0)
       (effects (font (size 1.27 1.27)) hide)
     )
@@
     )
     (path "/00000000-0000-0000-0000-00005fc468f3"
-      (reference "J4") (unit 1) (value "FLOPPY") (footprint "Connector_PinHeader_2.54mm:PinHeader_2x17_P2.54mm_Horizontal")
+      (reference "J4") (unit 1) (value "FLOPPY") (footprint "Connector_IDC:IDC-Header_2x17_P2.54mm_Vertical")
     )
     (path "/ebd9fdfc-3919-4a03-8180-54d97bd03282"
-      (reference "SW1") (unit 1) (value "SW_DPDT_x2") (footprint "")
+      (reference "SW1") (unit 1) (value "SW_DPDT_x2") (footprint "Button_Switch_THT:SW_CuK_JS202011AQN_DPDT_Angled")
     )
     (path "/60153e7c-7d60-42d1-a9fe-98c5063cb180"
-      (reference "SW1") (unit 2) (value "SW_DPDT_x2") (footprint "")
+      (reference "SW1") (unit 2) (value "SW_DPDT_x2") (footprint "Button_Switch_THT:SW_CuK_JS202011AQN_DPDT_Angled")
     )
     (path "/00000000-0000-0000-0000-00005fc363e4"
