File: external_floppy/floppy.kicad_sch (KiCad schematic)
At the start: 13 parts, among them J1 12VDC, J2 FLOPPY_PWR, J3 ADAPTER, J4 FLOPPY, SW1 SW_DPDT_x2, U1 L7805

Commit message: a
Parts:
- gave numbers to parts that had none: 4
Connections:
- net +5V: no longer J3.15 (Pin_15)
- no-connect marks 4 -> 5
Changed lines of the file:
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@@
   (junction (at 134.62 82.55) (diameter 0.9144) (color 0 0 0 0))
   (junction (at 134.62 85.09) (diameter 0.9144) (color 0 0 0 0))
+  (no_connect (at 92.71 87.63))
+  (no_connect (at 134.62 44.45))
+  (no_connect (at 121.92 59.69))
   (no_connect (at 121.92 46.99))
-  (no_connect (at 121.92 59.69))
-  (no_connect (at 134.62 44.45))
   (no_connect (at 121.92 49.53))
   (wire (pts (xy 26.67 63.5) (xy 26.67 60.96))
@@
     (effects (font (size 1.27 1.27)) (justify left bottom))
   )
-  (label "+5V" (at 92.71 87.63 0)
-    (effects (font (size 1.27 1.27)) (justify left bottom))
-  )
   (label "FLOPPY_DISKCHANGE" (at 121.92 44.45 180)
     (effects (font (size 1.27 1.27)) (justify right bottom))
@@
   (symbol (lib_id "power:GND") (at 113.03 133.35 0) (unit 1)
     (in_bom yes) (on_board yes)
-    (property "Reference" "#PWR?" (id 0) (at 113.03 139.7 0)
+    (property "Reference" "#PWR0104" (id 0) (at 113.03 139.7 0)
       (effects (font (size 1.27 1.27)) hide)
     )
@@
   (symbol (lib_id "Mechanical:MountingHole_Pad") (at 105.41 130.81 0) (unit 1)
     (in_bom yes) (on_board yes)
-    (property "Reference" "H?" (id 0) (at 109.22 129.54 0)
+    (property "Reference" "H1" (id 0) (at 109.22 129.54 0)
       (effects (font (size 1.27 1.27)) (justify left))
     )
@@
   (symbol (lib_id "Mechanical:MountingHole_Pad") (at 110.49 130.81 0) (unit 1)
     (in_bom yes) (on_board yes)
-    (property "Reference" "H?" (id 0) (at 114.3 129.54 0)
+    (property "Reference" "H2" (id 0) (at 114.3 129.54 0)
       (effects (font (size 1.27 1.27)) (justify left))
     )
@@
   (symbol (lib_id "Mechanical:MountingHole_Pad") (at 115.57 130.81 0) (unit 1)
     (in_bom yes) (on_board yes)
-    (property "Reference" "H?" (id 0) (at 119.38 129.54 0)
+    (property "Reference" "H3" (id 0) (at 119.38 129.54 0)
       (effects (font (size 1.27 1.27)) (justify left))
     )
@@
   (symbol (lib_id "Mechanical:MountingHole_Pad") (at 120.65 130.81 0) (unit 1)
     (in_bom yes) (on_board yes)
-    (property "Reference" "H?" (id 0) (at 124.46 129.54 0)
+    (property "Reference" "H4" (id 0) (at 124.46 129.54 0)
       (effects (font (size 1.27 1.27)) (justify left))
     )
@@
     )
     (path "/86c8debe-a504-4f15-b922-97104be1137e"
-      (reference "#PWR?") (unit 1) (value "GND") (footprint "")
+      (reference "#PWR0104") (unit 1) (value "GND") (footprint "")
     )
     (path "/00000000-0000-0000-0000-00005fc399bb"
@@
     )
     (path "/8d913606-4842-4a06-8920-27df9773221c"
-      (reference "H?") (unit 1) (value "MountingHole_Pad") (footprint "MountingHole:MountingHole_3.2mm_M3_DIN965_Pad_TopBottom")
+      (reference "H1") (unit 1) (value "MountingHole_Pad") (footprint "MountingHole:MountingHole_3.2mm_M3_DIN965_Pad_TopBottom")
+    )
+    (path "/ef780470-5014-4465-9c06-f868cd7bedd3"
+      (reference "H2") (unit 1) (value "MountingHole_Pad") (footprint "MountingHole:MountingHole_3.2mm_M3_DIN965_Pad_TopBottom")
     )
     (path "/cc995442-67f0-4be6-ba09-42302e9e6530"
-      (reference "H?") (unit 1) (value "MountingHole_Pad") (footprint "MountingHole:MountingHole_3.2mm_M3_DIN965_Pad_TopBottom")
+      (reference "H3") (unit 1) (value "MountingHole_Pad") (footprint "MountingHole:MountingHole_3.2mm_M3_DIN965_Pad_TopBottom")
     )
     (path "/d19e5e46-d244-4a0a-9c50-ce64a47de76d"
-      (reference "H?") (unit 1) (value "MountingHole_Pad") (footprint "MountingHole:MountingHole_3.2mm_M3_DIN965_Pad_TopBottom")
-    )
-    (path "/ef780470-5014-4465-9c06-f868cd7bedd3"
-      (reference "H?") (unit 1) (value "MountingHole_Pad") (footprint "MountingHole:MountingHole_3.2mm_M3_DIN965_Pad_TopBottom")
+      (reference "H4") (unit 1) (value "MountingHole_Pad") (footprint "MountingHole:MountingHole_3.2mm_M3_DIN965_Pad_TopBottom")
     )
     (path "/00000000-0000-0000-0000-00005fc2b4e0"
