File: external_floppy/floppy.kicad_sch (KiCad schematic)
At the start: 13 parts, among them J1 12VDC, J2 FLOPPY_PWR, J3 ADAPTER, J4 FLOPPY, SW1 SW_DPDT_x2, U1 L7805

Commit message: a
Connections:
- net FLOPPY_SELECT_A: now also SW1.2 (B); no longer SW1.1 (A), SW1.6 (C)
- net FLOPPY_SELECT_B: now also SW1.5 (B); no longer SW1.3 (C), SW1.4 (A)
- net F_INSEL_A: now also SW1.1 (A), SW1.6 (C); no longer SW1.2 (B)
- net F_INSEL_B: now also SW1.3 (C), SW1.4 (A); no longer SW1.5 (B)
Changed lines of the file:
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@@
   (junction (at 134.62 82.55) (diameter 0.9144) (color 0 0 0 0))
   (junction (at 134.62 85.09) (diameter 0.9144) (color 0 0 0 0))
-  (no_connect (at 92.71 87.63))
-  (no_connect (at 134.62 44.45))
-  (no_connect (at 121.92 59.69))
   (no_connect (at 121.92 46.99))
   (no_connect (at 121.92 49.53))
+  (no_connect (at 121.92 59.69))
+  (no_connect (at 134.62 44.45))
+  (no_connect (at 92.71 87.63))
   (wire (pts (xy 26.67 63.5) (xy 26.67 60.96))
     (stroke (width 0) (type solid) (color 0 0 0 0))
@@
     (stroke (width 0) (type solid) (color 0 0 0 0))
   )
-  (label "F_INSEL_A" (at 36.83 113.03 180)
-    (effects (font (size 1.27 1.27)) (justify right bottom))
-  )
-  (label "F_INSEL_B" (at 36.83 127 180)
-    (effects (font (size 1.27 1.27)) (justify right bottom))
-  )
-  (label "FLOPPY_SELECT_A" (at 46.99 110.49 0)
+  (label "F_INSEL_A" (at 36.83 110.49 180)
+    (effects (font (size 1.27 1.27)) (justify right bottom))
+  )
+  (label "F_INSEL_B" (at 36.83 115.57 180)
+    (effects (font (size 1.27 1.27)) (justify right bottom))
+  )
+  (label "F_INSEL_B" (at 36.83 124.46 180)
+    (effects (font (size 1.27 1.27)) (justify right bottom))
+  )
+  (label "F_INSEL_A" (at 36.83 129.54 180)
+    (effects (font (size 1.27 1.27)) (justify right bottom))
+  )
+  (label "FLOPPY_SELECT_A" (at 46.99 113.03 0)
     (effects (font (size 1.27 1.27)) (justify left bottom))
   )
-  (label "FLOPPY_SELECT_B" (at 46.99 115.57 0)
-    (effects (font (size 1.27 1.27)) (justify left bottom))
-  )
-  (label "FLOPPY_SELECT_B" (at 46.99 124.46 0)
-    (effects (font (size 1.27 1.27)) (justify left bottom))
-  )
-  (label "FLOPPY_SELECT_A" (at 46.99 129.54 0)
+  (label "FLOPPY_SELECT_B" (at 46.99 127 0)
     (effects (font (size 1.27 1.27)) (justify left bottom))
   )
@@
     )
   )
-  (symbol (lib_id "Switch:SW_DPDT_x2") (at 41.91 113.03 0) (unit 1)
+  (symbol (lib_id "Switch:SW_DPDT_x2") (at 41.91 113.03 0) (mirror y) (unit 1)
     (in_bom yes) (on_board yes)
     (property "Reference" "SW1" (id 0) (at 41.91 105.41 0))
@@
     )
   )
-  (symbol (lib_id "Switch:SW_DPDT_x2") (at 41.91 127 0) (unit 2)
+  (symbol (lib_id "Switch:SW_DPDT_x2") (at 41.91 127 0) (mirror y) (unit 2)
     (in_bom yes) (on_board yes)
     (property "Reference" "SW1" (id 0) (at 41.91 119.38 0))
