File: external_floppy/floppy.kicad_pcb (KiCad board)
At the start: 2 copper layers, 10 parts, among them J1 12VDC, J3 ADAPTER, J4 FLOPPY, J5 ADAPTER, J6 ATARI, SW1 SW_DPDT_x2, U1 L7805

Commit message: a
Parts:
- J4: footprint Connector_PinHeader_2.54mm:PinHeader_2x17_P2.54mm_Horizontal -> Connector_IDC:IDC-Header_2x17_P2.54mm_Vertical
- moved D1 111.8 mm to (38.1, 50.8)
- moved J1 105.5 mm to (63.5, 50.8), turned to -90 degrees
- moved U1 83.8 mm to (63.5, 63.5), turned to 180 degrees
- moved C2 60.6 mm to (76.2, 63.5)
- moved C1 56.8 mm to (76.2, 76.2)
- moved J3 47.7 mm to (83.8, 50.8), turned to 90 degrees
- moved SW1 40.7 mm to (127.0, 50.8), turned to 180 degrees
- moved J4 33.7 mm to (114.3, 101.6), turned to -90 degrees

Commit message: a
Parts:
- removed J5: ADAPTER, Connector_IDC:IDC-Header_2x08_P2.54mm_Vertical
- removed J6: ATARI, parts:DIN14
- added H1: MountingHole_Pad, MountingHole:MountingHole_3.2mm_M3_DIN965_Pad_TopBottom, F.Cu at (124.5, 67.3)
- added H2: MountingHole_Pad, MountingHole:MountingHole_3.2mm_M3_DIN965_Pad_TopBottom, F.Cu at (35.6, 104.1)
- added H3: MountingHole_Pad, MountingHole:MountingHole_3.2mm_M3_DIN965_Pad_TopBottom, F.Cu at (124.5, 104.1)
- added H4: MountingHole_Pad, MountingHole:MountingHole_3.2mm_M3_DIN965_Pad_TopBottom, F.Cu at (35.6, 67.3)
- added J2: FLOPPY_PWR, Connector_Molex:Molex_KK-254_AE-6410-04A_1x04_P2.54mm_Vertical, F.Cu at (55.2, 102.9)
- moved SW1 59.1 mm to (70.5, 67.9)
- moved C2 38.6 mm to (55.2, 95.9), turned to 90 degrees
- moved D1 32.5 mm to (47.6, 81.9)
- moved U1 28.4 mm to (47.6, 87.0)
- moved J1 27.3 mm to (55.2, 76.8)
- moved J3 25.5 mm to (81.3, 76.2)
- moved C1 22.5 mm to (64.1, 95.2), turned to 90 degrees
Other:
- board outline added: 96.5 x 44.5 mm

Commit message: a
Parts:
- moved SW1 44.3 mm to (114.8, 68.3)
Connections:
- J3 pad 15: +5V -> no_connect_35
- J4 pad 1: no_connect_35 -> no_connect_36
- J4 pad 14: no_connect_36 -> no_connect_37
- J4 pad 4: no_connect_37 -> no_connect_38
- J4 pad 6: no_connect_38 -> no_connect_39
Changed lines of the file:
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@@
   (net 23 "no_connect_37")
   (net 24 "no_connect_35")
+  (net 25 "no_connect_39")
   (footprint "Package_TO_SOT_THT:TO-220-3_Horizontal_TabDown" (layer "F.Cu")
     (at 47.625 86.995 180)
@@
   )
   (footprint "Button_Switch_THT:SW_CuK_JS202011AQN_DPDT_Angled" (layer "F.Cu")
-    (at 70.485 67.945 180)
+    (at 114.75 68.3 180)
     (descr "CuK sub miniature slide switch, JS series, DPDT, right angle, http://www.ckswitches.com/media/1422/js.pdf")
     (tags "switch DPDT")
@@
       (net 5 "/FLOPPY_READY") (pinfunction "Pin_14"))
     (pad "15" thru_hole circle (at 0 17.78 90) (size 1.7 1.7) (drill 1) (layers *.Cu *.Mask)
-      (net 3 "+5V") (pinfunction "Pin_15"))
+      (net 24 "no_connect_35") (pinfunction "Pin_15"))
     (pad "16" thru_hole circle (at 2.54 17.78 90) (size 1.7 1.7) (drill 1) (layers *.Cu *.Mask)
       (net 1 "GND") (pinfunction "Pin_16"))
@@
     (fp_line (start -3.18 18.27) (end -1.98 18.27) (layer "F.Fab") (width 0.1))
     (pad "1" thru_hole roundrect (at 0 0 270) (size 1.7 1.7) (drill 1) (layers *.Cu *.Mask) (roundrect_rratio 0.147059)
-      (net 24 "no_connect_35") (pinfunction "Pin_1"))
+      (net 19 "no_connect_36") (pinfunction "Pin_1"))
     (pad "2" thru_hole circle (at 2.54 0 270) (size 1.7 1.7) (drill 1) (layers *.Cu *.Mask)
       (net 18 "/FLOPPY_DISKCHANGE") (pinfunction "Pin_2"))
@@
       (net 1 "GND") (pinfunction "Pin_3"))
     (pad "4" thru_hole circle (at 2.54 2.54 270) (size 1.7 1.7) (drill 1) (layers *.Cu *.Mask)
-      (net 23 "no_connect_37") (pinfunction "Pin_4"))
+      (net 22 "no_connect_38") (pinfunction "Pin_4"))
     (pad "5" thru_hole circle (at 0 5.08 270) (size 1.7 1.7) (drill 1) (layers *.Cu *.Mask)
       (net 1 "GND") (pinfunction "Pin_5"))
     (pad "6" thru_hole circle (at 2.54 5.08 270) (size 1.7 1.7) (drill 1) (layers *.Cu *.Mask)
-      (net 22 "no_connect_38") (pinfunction "Pin_6"))
+      (net 25 "no_connect_39") (pinfunction "Pin_6"))
     (pad "7" thru_hole circle (at 0 7.62 270) (size 1.7 1.7) (drill 1) (layers *.Cu *.Mask)
       (net 1 "GND") (pinfunction "Pin_7"))
@@
       (net 1 "GND") (pinfunction "Pin_13"))
     (pad "14" thru_hole circle (at 2.54 15.24 270) (size 1.7 1.7) (drill 1) (layers *.Cu *.Mask)
-      (net 19 "no_connect_36") (pinfunction "Pin_14"))
+      (net 23 "no_connect_37") (pinfunction "Pin_14"))
     (pad "15" thru_hole circle (at 0 17.78 270) (size 1.7 1.7) (drill 1) (layers *.Cu *.Mask)
       (net 1 "GND") (pinfunction "Pin_15"))

Commit message: a
Connections:
- SW1 pad 1: /FLOPPY_SELECT_A -> /F_INSEL_A
- SW1 pad 2: /F_INSEL_A -> /FLOPPY_SELECT_A
- SW1 pad 3: /FLOPPY_SELECT_B -> /F_INSEL_B
- SW1 pad 4: /FLOPPY_SELECT_B -> /F_INSEL_B
- SW1 pad 5: /F_INSEL_B -> /FLOPPY_SELECT_B
- SW1 pad 6: /FLOPPY_SELECT_A -> /F_INSEL_A
Routing:
- net /FLOPPY_SIDE_SELECT: track 0.00 -> 60.4 mm
- net /FLOPPY_READY: track 0.00 -> 58.5 mm
- net /FLOPPY_WRITE_PROTECT: track 0.00 -> 54.3 mm
- net /FLOPPY_READ_DATA: track 0.00 -> 53.2 mm
- net /FLOPPY_WRITE_DATA: track 0.00 -> 49.5 mm
- net /F_INSEL_A: track 0.00 -> 46.6 mm
- net /FLOPPY_DISKCHANGE: track 0.00 -> 45.7 mm
- net /F_INSEL_B: track 0.00 -> 45.7 mm
- net /FLOPPY_INDEX: track 0.00 -> 43.0 mm
- net /FLOPPY_TRACK_00: track 0.00 -> 42.9 mm
- net /FLOPPY_WRITE_GATE: track 0.00 -> 41.9 mm
- net /FLOPPY_STEP: track 0.00 -> 41.5 mm
- net /FLOPPY_MOTOR_ON: track 0.00 -> 35.8 mm
- net /FLOPPY_STEP_DIRECTION: track 0.00 -> 34.7 mm
- net +12V: track 0.00 -> 33.2 mm
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- added copper zone on B.Cu, net GND
- added copper zone on F.Cu, net GND
Other:
- board text added: "DRIVE SELECT 0 / 1"
- board text added: "NORMAL"
- board text added: "REVERSED"

Commit message: a
Routing:
- net /FLOPPY_WRITE_PROTECT: track 54.3 -> 51.3 mm
- net /FLOPPY_READ_DATA: track 53.2 -> 50.6 mm
- net /FLOPPY_SIDE_SELECT: track 60.4 -> 58.3 mm

Commit message: a
Routing:
- net /FLOPPY_SIDE_SELECT: track 58.3 -> 55.6 mm
- net /FLOPPY_READY: track 58.9 -> 56.5 mm
- net /FLOPPY_READ_DATA: track 50.6 -> 49.9 mm
Changed lines of the file:
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@@
   (segment (start 51.435 95.885) (end 55.245 95.885) (width 0.4) (layer "F.Cu") (net 3))
   (segment (start 55.245 76.835) (end 55.245 81.915) (width 0.4) (layer "F.Cu") (net 4))
-  (segment (start 81.251467 68.149991) (end 74.949999 74.451459) (width 0.4) (layer "F.Cu") (net 5))
+  (segment (start 81.35001 68.89999) (end 81.425739 68.89999) (width 0.4) (layer "F.Cu") (net 5))
+  (segment (start 81.35001 68.89999) (end 92.14999 68.89999) (width 0.4) (layer "F.Cu") (net 5))
   (segment (start 96.52 73.02) (end 96.52 73.66) (width 0.4) (layer "F.Cu") (net 5))
-  (segment (start 96.52 73.66) (end 96.52 70.921458) (width 0.4) (layer "F.Cu") (net 5))
-  (segment (start 93.748532 68.14999) (end 81.251467 68.149991) (width 0.4) (layer "F.Cu") (net 5))
-  (segment (start 74.949999 74.451459) (end 74.949999 102.850001) (width 0.4) (layer "F.Cu") (net 5))
-  (segment (start 96.52 70.921458) (end 93.748532 68.14999) (width 0.4) (layer "F.Cu") (net 5))
-  (segment (start 74.949999 102.850001) (end 73.66 104.14) (width 0.4) (layer "F.Cu") (net 5))
+  (segment (start 74.949999 102.850001) (end 74.949999 75.300001) (width 0.4) (layer "F.Cu") (net 5))
+  (segment (start 73.66 104.14) (end 74.949999 102.850001) (width 0.4) (layer "F.Cu") (net 5))
+  (segment (start 74.949999 75.300001) (end 81.35001 68.89999) (width 0.4) (layer "F.Cu") (net 5))
+  (segment (start 92.14999 68.89999) (end 96.52 73.27) (width 0.4) (layer "F.Cu") (net 5))
+  (segment (start 96.52 73.27) (end 96.52 73.66) (width 0.4) (layer "F.Cu") (net 5))
   (segment (start 78.74 104.14) (end 78.74 103.450002) (width 0.4) (layer "F.Cu") (net 6))
-  (segment (start 91.85001 70.10001) (end 82.14999 70.10001) (width 0.4) (layer "F.Cu") (net 6))
-  (segment (start 93.98 73.66) (end 93.98 72.23) (width 0.4) (layer "F.Cu") (net 6))
+  (segment (start 93.98 73.66) (end 93.98 73.23) (width 0.4) (layer "F.Cu") (net 6))
+  (segment (start 93.98 73.23) (end 91 70.25) (width 0.4) (layer "F.Cu") (net 6))
+  (segment (start 82 70.25) (end 78.75 73.5) (width 0.4) (layer "F.Cu") (net 6))
+  (segment (start 78.75 73.5) (end 78.75 93.25) (width 0.4) (layer "F.Cu") (net 6))
   (segment (start 79.990001 102.200001) (end 79.990001 94.490001) (width 0.4) (layer "F.Cu") (net 6))
+  (segment (start 78.75 93.25) (end 80 94.5) (width 0.4) (layer "F.Cu") (net 6))
+  (segment (start 91 70.25) (end 82 70.25) (width 0.4) (layer "F.Cu") (net 6))
   (segment (start 78.74 103.450002) (end 79.990001 102.200001) (width 0.4) (layer "F.Cu") (net 6))
-  (segment (start 82.14999 70.10001) (end 78.75 73.5) (width 0.4) (layer "F.Cu") (net 6))
-  (segment (start 78.75 93.25) (end 80 94.5) (width 0.4) (layer "F.Cu") (net 6))
-  (segment (start 93.98 72.23) (end 91.85001 70.10001) (width 0.4) (layer "F.Cu") (net 6))
-  (segment (start 78.75 73.5) (end 78.75 93.25) (width 0.4) (layer "F.Cu") (net 6))
-  (segment (start 89.748534 71.80999) (end 91.44 73.501456) (width 0.4) (layer "F.Cu") (net 7))
-  (segment (start 85.070001 102.889999) (end 85.070001 97.570001) (width 0.4) (layer "F.Cu") (net 7))
-  (segment (start 82.530001 73.099997) (end 83.820009 71.809989) (width 0.4) (layer "F.Cu") (net 7))
-  (segment (start 82.530001 95.030001) (end 82.530001 73.099997) (width 0.4) (layer "F.Cu") (net 7))
-  (segment (start 91.44 73.501456) (end 91.44 73.66) (width 0.4) (layer "F.Cu") (net 7))
-  (segment (start 83.820009 71.809989) (end 89.748534 71.80999) (width 0.4) (layer "F.Cu") (net 7))
-  (segment (start 85.070001 97.570001) (end 82.530001 95.030001) (width 0.4) (layer "F.Cu") (net 7))
-  (segment (start 83.82 104.14) (end 85.070001 102.889999) (width 0.4) (layer "F.Cu") (net 7))
+  (segment (start 85.070001 102.889999) (end 83.82 104.14) (width 0.4) (layer "F.Cu") (net 7))
+  (segment (start 83.879998 71.75) (end 83.820009 71.809989) (width 0.4) (layer "F.Cu") (net 7))
+  (segment (start 90 71.75) (end 83.879998 71.75) (width 0.4) (layer "F.Cu") (net 7))
+  (segment (start 91.44 73.19) (end 90 71.75) (width 0.4) (layer "F.Cu") (net 7))
+  (segment (start 85.070001 97.570001) (end 85.070001 102.889999) (width 0.4) (layer "F.Cu") (net 7))
+  (segment (start 82.530001 73.099997) (end 82.530001 95.030001) (width 0.4) (layer "F.Cu") (net 7))
+  (segment (start 83.879998 71.75) (end 82.530001 73.099997) (width 0.4) (layer "F.Cu") (net 7))
+  (segment (start 82.530001 95.030001) (end 85.070001 97.570001) (width 0.4) (layer "F.Cu") (net 7))
+  (segment (start 91.44 73.66) (end 91.44 73.19) (width 0.4) (layer "F.Cu") (net 7))
   (segment (start 100.310001 101.060001) (end 100.310001 104.740001) (width 0.4) (layer "F.Cu") (net 8))
   (segment (start 97.800002 107.25) (end 92.01 107.25) (width 0.4) (layer "F.Cu") (net 8))
@@
   (segment (start 80.02999 77.27999) (end 102.75 100) (width 0.4) (layer "B.Cu") (net 11))
   (segment (start 80.02999 74.91001) (end 80.02999 77.27999) (width 0.4) (layer "B.Cu") (net 11))
-  (segment (start 77.450001 72.799999) (end 81.5 68.75) (width 0.4) (layer "F.Cu") (net 12))
-  (segment (start 77.450001 102.889999) (end 77.450001 72.799999) (width 0.4) (layer "F.Cu") (net 12))
-  (segment (start 95.269999 70.519999) (end 95.269999 74.949999) (width 0.4) (layer "F.Cu") (net 12))
-  (segment (start 81.5 68.75) (end 93.5 68.75) (width 0.4) (layer "F.Cu") (net 12))
-  (segment (start 93.5 68.75) (end 95.269999 70.519999) (width 0.4) (layer "F.Cu") (net 12))
+  (segment (start 91.75 69.5) (end 95.269999 73.019999) (width 0.4) (layer "F.Cu") (net 12))
+  (segment (start 77.450001 102.889999) (end 77.450001 73.799999) (width 0.4) (layer "F.Cu") (net 12))
+  (segment (start 81.75 69.5) (end 91.75 69.5) (width 0.4) (layer "F.Cu") (net 12))
+  (segment (start 77.450001 73.799999) (end 81.75 69.5) (width 0.4) (layer "F.Cu") (net 12))
   (segment (start 95.269999 74.949999) (end 96.52 76.2) (width 0.4) (layer "F.Cu") (net 12))
   (segment (start 76.2 104.14) (end 77.450001 102.889999) (width 0.4) (layer "F.Cu") (net 12))
+  (segment (start 95.269999 73.019999) (end 95.269999 74.949999) (width 0.4) (layer "F.Cu") (net 12))
+  (segment (start 82.530001 102.889999) (end 81.28 104.14) (width 0.4) (layer "F.Cu") (net 13))
+  (segment (start 82.098542 71) (end 80 73.098542) (width 0.4) (layer "F.Cu") (net 13))
+  (segment (start 90.630002 71) (end 82.098542 71) (width 0.4) (layer "F.Cu") (net 13))
   (segment (start 93.98 76.2) (end 92.729999 74.949999) (width 0.4) (layer "F.Cu") (net 13))
-  (segment (start 90.630002 71) (end 82.098542 71) (width 0.4) (layer "F.Cu") (net 13))
+  (segment (start 82.530001 95.878543) (end 82.530001 102.889999) (width 0.4) (layer "F.Cu") (net 13))
   (segment (start 92.729999 74.949999) (end 92.729999 73.099997) (width 0.4) (layer "F.Cu") (net 13))
-  (segment (start 82.530001 102.889999) (end 81.28 104.14) (width 0.4) (layer "F.Cu") (net 13))
-  (segment (start 82.530001 95.878543) (end 82.530001 102.889999) (width 0.4) (layer "F.Cu") (net 13))
   (segment (start 92.729999 73.099997) (end 90.630002 71) (width 0.4) (layer "F.Cu") (net 13))
   (segment (start 90.630002 71) (end 90 71) (width 0.4) (layer "F.Cu") (net 13))
+  (segment (start 80 93.348542) (end 82.530001 95.878543) (width 0.4) (layer "F.Cu") (net 13))
   (segment (start 80 73.098542) (end 80 93.348542) (width 0.4) (layer "F.Cu") (net 13))
-  (segment (start 82.098542 71) (end 80 73.098542) (width 0.4) (layer "F.Cu") (net 13))
-  (segment (start 80 93.348542) (end 82.530001 95.878543) (width 0.4) (layer "F.Cu") (net 13))
   (segment (start 90.150001 74.260001) (end 90.150001 73.059999) (width 0.4) (layer "F.Cu") (net 14))
   (segment (start 91.44 76.2) (end 91.44 75.55) (width 0.4) (layer "F.Cu") (net 14))

Commit message: a
Routing:
- net /FLOPPY_WRITE_GATE: track 41.9 -> 58.4 mm
- net /FLOPPY_MOTOR_ON: track 35.8 -> 51.6 mm
- net /FLOPPY_STEP_DIRECTION: track 34.7 -> 50.0 mm
- net /FLOPPY_TRACK_00: track 43.2 -> 56.8 mm
- net /FLOPPY_STEP: track 41.5 -> 55.0 mm
- net /FLOPPY_WRITE_PROTECT: track 51.3 -> 61.9 mm
- net /FLOPPY_READ_DATA: track 49.9 -> 60.3 mm
- net /FLOPPY_SIDE_SELECT: track 55.6 -> 65.3 mm
- net /FLOPPY_READY: track 56.5 -> 64.5 mm
- net /FLOPPY_DISKCHANGE: track 45.7 -> 49.7 mm
- net /FLOPPY_WRITE_DATA: track 49.5 -> 53.4 mm
- net /FLOPPY_INDEX: track 43.0 -> 41.0 mm

Commit message: a
Parts:
- J2: footprint Connector_Molex:Molex_KK-254_AE-6410-04A_1x04_P2.54mm_Vertical -> Connector_PinHeader_2.54mm:PinHeader_1x04_P2.54mm_Vertical
- moved J2 3.77 mm to (55.2, 99.1), turned to 90 degrees
- moved C2 3.14 mm to (55.2, 92.8)
- moved C1 2.61 mm to (63.4, 92.8)
Routing:
- net +12V: track 33.2 -> 5.08 mm
- net +5V: track 23.4 -> 0.00 mm
Other:
- outline, holes or cut-outs redrawn
