File: external_floppy/floppy.kicad_pcb (KiCad board)
At the start: 2 copper layers, 96.5 x 44.5 mm, 13 parts, among them J1 12VDC, J2 FLOPPY_PWR, J3 ADAPTER, J4 FLOPPY, SW1 SW_DPDT_x2, U1 L7805

Commit message: a
Parts:
- C1: footprint Capacitor_THT:C_Radial_D10.0mm_H12.5mm_P5.00mm -> Capacitor_THT:CP_Radial_D10.0mm_P5.00mm
Routing:
- net +12V: track 5.08 -> 29.8 mm
- net +5V: track 0.00 -> 22.6 mm
- net /FLOPPY_SELECT_B: track 32.1 -> 33.2 mm
Other:
- board text added: "+12V"
- board text added: "+5V"
- board text added: "GND"
