File: acsi_to_scsi.kicad_sch (KiCad schematic)
At the start: 15 parts, among them J1 SCSI, U1 74ALS573, U10 74LS02, U11 74ALS74, U2 74ALS540, U3 74ALS540, U4 74LS01, U5 74ALS74, U6 74ALS08, U7 74ALS85, U8 74LS04, U9 74LS08

Commit message: a
Parts:
- added R?: 1k, symbol Device:R
Connections:
- net GND: now also SW?.4, SW?.5, SW?.6, U10.8, U10.9, U7.9 (B0), U9.1, U9.2, U9.4, U9.5
- net VCC: now also J1.26 (Pin_26), R?.1
- net at U8.5: now also J1.48 (Pin_48)
- net at U8.8: now also J1.40 (Pin_40)
- net at U9.10: now also J1.50 (Pin_50), U9.9
- net at J1.32 (Pin_32): now also R?.2
- no-connect marks 1 -> 14
Other:
- moved on the sheet: J1, U10A, U10C, U10D, U4A, U4D, U5A, U5B, U8A, U8C, U8D, U9A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

Commit message: a
Connections:
- net GND: now also U1.1 (OE), U1.10 (GND)
- net at U2.1 (~G1): now also J1.36 (Pin_36), U3.1 (~G1)
Other:
- moved on the sheet: U8B
Changed lines of the file:
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@@
   (junction (at 63.5 69.85) (diameter 0.9144) (color 0 0 0 0))
   (junction (at 66.04 67.31) (diameter 0.9144) (color 0 0 0 0))
+  (junction (at 81.28 100.33) (diameter 0.9144) (color 0 0 0 0))
   (junction (at 119.38 137.16) (diameter 0.9144) (color 0 0 0 0))
   (junction (at 119.38 139.7) (diameter 0.9144) (color 0 0 0 0))
@@
   (junction (at 138.43 127) (diameter 0.9144) (color 0 0 0 0))
   (junction (at 138.43 140.97) (diameter 0.9144) (color 0 0 0 0))
+  (junction (at 179.07 58.42) (diameter 0.9144) (color 0 0 0 0))
   (junction (at 293.37 207.01) (diameter 0.9144) (color 0 0 0 0))
   (junction (at 312.42 85.09) (diameter 0.9144) (color 0 0 0 0))
@@
     (stroke (width 0) (type solid) (color 0 0 0 0))
   )
+  (wire (pts (xy 68.58 100.33) (xy 68.58 92.71))
+    (stroke (width 0) (type solid) (color 0 0 0 0))
+  )
+  (wire (pts (xy 81.28 100.33) (xy 68.58 100.33))
+    (stroke (width 0) (type solid) (color 0 0 0 0))
+  )
   (wire (pts (xy 93.98 67.31) (xy 96.52 67.31))
     (stroke (width 0) (type solid) (color 0 0 0 0))
@@
     (stroke (width 0) (type solid) (color 0 0 0 0))
   )
-  (wire (pts (xy 96.52 67.31) (xy 96.52 33.02))
+  (wire (pts (xy 96.52 67.31) (xy 96.52 22.86))
     (stroke (width 0) (type solid) (color 0 0 0 0))
   )
@@
     (stroke (width 0) (type solid) (color 0 0 0 0))
   )
-  (wire (pts (xy 99.06 30.48) (xy 193.04 30.48))
-    (stroke (width 0) (type solid) (color 0 0 0 0))
-  )
-  (wire (pts (xy 99.06 69.85) (xy 99.06 30.48))
+  (wire (pts (xy 99.06 20.32) (xy 193.04 20.32))
+    (stroke (width 0) (type solid) (color 0 0 0 0))
+  )
+  (wire (pts (xy 99.06 69.85) (xy 99.06 20.32))
     (stroke (width 0) (type solid) (color 0 0 0 0))
   )
@@
     (stroke (width 0) (type solid) (color 0 0 0 0))
   )
-  (wire (pts (xy 101.6 27.94) (xy 190.5 27.94))
-    (stroke (width 0) (type solid) (color 0 0 0 0))
-  )
-  (wire (pts (xy 101.6 72.39) (xy 101.6 27.94))
+  (wire (pts (xy 101.6 17.78) (xy 190.5 17.78))
+    (stroke (width 0) (type solid) (color 0 0 0 0))
+  )
+  (wire (pts (xy 101.6 72.39) (xy 101.6 17.78))
     (stroke (width 0) (type solid) (color 0 0 0 0))
   )
@@
     (stroke (width 0) (type solid) (color 0 0 0 0))
   )
-  (wire (pts (xy 104.14 25.4) (xy 104.14 74.93))
+  (wire (pts (xy 104.14 15.24) (xy 104.14 74.93))
     (stroke (width 0) (type solid) (color 0 0 0 0))
   )
@@
     (stroke (width 0) (type solid) (color 0 0 0 0))
   )
-  (wire (pts (xy 106.68 22.86) (xy 106.68 77.47))
-    (stroke (width 0) (type solid) (color 0 0 0 0))
-  )
-  (wire (pts (xy 106.68 22.86) (xy 185.42 22.86))
+  (wire (pts (xy 106.68 12.7) (xy 106.68 77.47))
+    (stroke (width 0) (type solid) (color 0 0 0 0))
+  )
+  (wire (pts (xy 106.68 12.7) (xy 185.42 12.7))
     (stroke (width 0) (type solid) (color 0 0 0 0))
   )
@@
     (stroke (width 0) (type solid) (color 0 0 0 0))
   )
-  (wire (pts (xy 185.42 22.86) (xy 185.42 77.47))
+  (wire (pts (xy 168.91 58.42) (xy 179.07 58.42))
+    (stroke (width 0) (type solid) (color 0 0 0 0))
+  )
+  (wire (pts (xy 179.07 58.42) (xy 199.39 58.42))
+    (stroke (width 0) (type solid) (color 0 0 0 0))
+  )
+  (wire (pts (xy 179.07 90.17) (xy 179.07 58.42))
+    (stroke (width 0) (type solid) (color 0 0 0 0))
+  )
+  (wire (pts (xy 185.42 12.7) (xy 185.42 77.47))
     (stroke (width 0) (type solid) (color 0 0 0 0))
   )
@@
     (stroke (width 0) (type solid) (color 0 0 0 0))
   )
-  (wire (pts (xy 187.96 25.4) (xy 104.14 25.4))
-    (stroke (width 0) (type solid) (color 0 0 0 0))
-  )
-  (wire (pts (xy 187.96 74.93) (xy 187.96 25.4))
+  (wire (pts (xy 187.96 15.24) (xy 104.14 15.24))
+    (stroke (width 0) (type solid) (color 0 0 0 0))
+  )
+  (wire (pts (xy 187.96 74.93) (xy 187.96 15.24))
     (stroke (width 0) (type solid) (color 0 0 0 0))
   )
@@
     (stroke (width 0) (type solid) (color 0 0 0 0))
   )
-  (wire (pts (xy 190.5 27.94) (xy 190.5 72.39))
+  (wire (pts (xy 190.5 17.78) (xy 190.5 72.39))
     (stroke (width 0) (type solid) (color 0 0 0 0))
   )
@@
     (stroke (width 0) (type solid) (color 0 0 0 0))
   )
-  (wire (pts (xy 193.04 30.48) (xy 193.04 69.85))
+  (wire (pts (xy 193.04 20.32) (xy 193.04 69.85))
     (stroke (width 0) (type solid) (color 0 0 0 0))
   )
@@
     (stroke (width 0) (type solid) (color 0 0 0 0))
   )
-  (wire (pts (xy 195.58 33.02) (xy 96.52 33.02))
-    (stroke (width 0) (type solid) (color 0 0 0 0))
-  )
-  (wire (pts (xy 195.58 67.31) (xy 195.58 33.02))
+  (wire (pts (xy 195.58 22.86) (xy 96.52 22.86))
+    (stroke (width 0) (type solid) (color 0 0 0 0))
+  )
+  (wire (pts (xy 195.58 67.31) (xy 195.58 22.86))
     (stroke (width 0) (type solid) (color 0 0 0 0))
   )
@@
     (stroke (width 0) (type solid) (color 0 0 0 0))
   )
+  (wire (pts (xy 386.08 90.17) (xy 179.07 90.17))
+    (stroke (width 0) (type solid) (color 0 0 0 0))
+  )
+  (wire (pts (xy 386.08 110.49) (xy 386.08 90.17))
+    (stroke (width 0) (type solid) (color 0 0 0 0))
+  )
   (wire (pts (xy 386.08 125.73) (xy 401.32 125.73))
     (stroke (width 0) (type solid) (color 0 0 0 0))
@@
   )
   (wire (pts (xy 401.32 87.63) (xy 363.22 87.63))
+    (stroke (width 0) (type solid) (color 0 0 0 0))
+  )
+  (wire (pts (xy 401.32 110.49) (xy 386.08 110.49))
     (stroke (width 0) (type solid) (color 0 0 0 0))
   )
@@
   )
   (text "ORIGINALLY 74F540\nBUT MODERN ALS SHOULD BE\nFAST ENOUGH (I HOPE)"
-    (at 147.32 50.8 0)
+    (at 143.51 93.98 0)
     (effects (font (size 1.27 1.27)) (justify left bottom))
   )
@@
     )
     (property "Datasheet" "" (id 3) (at 389.89 97.79 0)
+      (effects (font (size 1.27 1.27)) hide)
+    )
+  )
+  (symbol (lib_id "power:GND") (at 81.28 100.33 0) (unit 1)
+    (in_bom yes) (on_board yes)
+    (property "Reference" "#PWR?" (id 0) (at 81.28 106.68 0)
+      (effects (font (size 1.27 1.27)) hide)
+    )
+    (property "Value" "GND" (id 1) (at 82.55 105.41 0))
+    (property "Footprint" "" (id 2) (at 81.28 100.33 0)
+      (effects (font (size 1.27 1.27)) hide)
+    )
+    (property "Datasheet" "" (id 3) (at 81.28 100.33 0)
       (effects (font (size 1.27 1.27)) hide)
     )
@@
     )
   )
-  (symbol (lib_id "74xx:74LS04") (at 67.31 107.95 0) (unit 2)
-    (in_bom yes) (on_board yes)
-    (property "Reference" "U8" (id 0) (at 67.31 99.8982 0))
-    (property "Value" "74LS04" (id 1) (at 67.31 102.2096 0))
-    (property "Footprint" "" (id 2) (at 67.31 107.95 0)
-      (effects (font (size 1.27 1.27)) hide)
-    )
-    (property "Datasheet" "http://www.ti.com/lit/gpn/sn74LS04" (id 3) (at 67.31 107.95 0)
+  (symbol (lib_id "74xx:74LS04") (at 64.77 107.95 0) (unit 2)
+    (in_bom yes) (on_board yes)
+    (property "Reference" "U8" (id 0) (at 64.77 99.8982 0))
+    (property "Value" "74LS04" (id 1) (at 64.77 102.2096 0))
+    (property "Footprint" "" (id 2) (at 64.77 107.95 0)
+      (effects (font (size 1.27 1.27)) hide)
+    )
+    (property "Datasheet" "http://www.ti.com/lit/gpn/sn74LS04" (id 3) (at 64.77 107.95 0)
       (effects (font (size 1.27 1.27)) hide)
     )
@@
       (reference "#PWR?") (unit 1) (value "GND") (footprint "")
     )
+    (path "/58b6dc4f-6436-4473-82fa-1b206df4d314"
+      (reference "#PWR?") (unit 1) (value "GND") (footprint "")
+    )

Commit message: a
Connections:
- net GND: now also U10.7 (GND), U11.7 (GND), U4.7 (GND), U5.7 (GND), U6.7 (GND), U8.7 (GND), U9.7 (GND)
- net VCC: now also U10.14 (VCC), U11.14 (VCC), U4.14 (VCC), U5.14 (VCC), U6.14 (VCC), U8.14 (VCC), U9.14 (VCC)
Other:
- moved on the sheet: U10E, U11C, U4E, U5C, U6E, U8G, U9E

Commit message: a
Connections:
- net at U1.11 (Load): now also U9.11
- net at U2.19 (~G2): now also U7.3 (Ia=b), U8.4
- net A0: now reaches U7.10 (A0)
- net A0: now also J?.16 (Pin_16)
- net SEL: now reaches U9.12
- net SEL: now also J?.9 (Pin_9), U11.11 (C)
- net ACK: now reaches U9.13
- net ACK: now also J?.14 (Pin_14)
- net R/W: now reaches U8.3
- net R/W: now also J?.18 (Pin_18)
- no-connect marks 14 -> 13
Other:
- moved on the sheet: J1, J?, R?, U10C, U10E, U11B, U11C, U2, U4A, U4D, U4E, U5C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

Commit message: a
Connections:
- net DR: now reaches U4.1
- net DR: now also J?.19 (Pin_19)
Other:
- moved on the sheet: U11B, U4A, U8F
Changed lines of the file:
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@@
+    (stroke (width 0) (type solid) (color 0 0 0 0))
+  )
+  (wire (pts (xy 21.59 113.03) (xy 2.54 113.03))
+    (stroke (width 0) (type solid) (color 0 0 0 0))
+  )
+  (wire (pts (xy 21.59 208.28) (xy 21.59 113.03))
     (stroke (width 0) (type solid) (color 0 0 0 0))
   )
@@
     (stroke (width 0) (type solid) (color 0 0 0 0))
   )
-  (wire (pts (xy 26.67 139.7) (xy 26.67 193.04))
+  (wire (pts (xy 26.67 139.7) (xy 26.67 182.88))
     (stroke (width 0) (type solid) (color 0 0 0 0))
   )
@@
     (stroke (width 0) (type solid) (color 0 0 0 0))
   )
-  (wire (pts (xy 26.67 193.04) (xy 57.15 193.04))
+  (wire (pts (xy 26.67 182.88) (xy 57.15 182.88))
+    (stroke (width 0) (type solid) (color 0 0 0 0))
+  )
+  (wire (pts (xy 26.67 208.28) (xy 21.59 208.28))
     (stroke (width 0) (type solid) (color 0 0 0 0))
   )
@@
     (stroke (width 0) (type solid) (color 0 0 0 0))
   )
-  (text "U4C on orig\n" (at 41.656 217.932 180)
+  (text "U4C on orig\n" (at 39.116 198.882 180)
     (effects (font (size 1.27 1.27)) (justify right bottom))
   )
@@
     (effects (font (size 1.27 1.27)) (justify right bottom))
   )
+  (label "DR" (at 21.59 113.03 180)
+    (effects (font (size 1.27 1.27)) (justify right bottom))
+  )
   (symbol (lib_id "power:VCC") (at 233.68 234.95 0) (unit 1)
     (in_bom yes) (on_board yes)
@@
     )
   )
-  (symbol (lib_id "74xx:74LS04") (at -3.81 189.23 90) (unit 6)
-    (in_bom yes) (on_board yes)
-    (property "Reference" "U8" (id 0) (at -11.8618 189.23 0))
-    (property "Value" "74LS04" (id 1) (at -9.5504 189.23 0))
-    (property "Footprint" "" (id 2) (at -3.81 189.23 0)
-      (effects (font (size 1.27 1.27)) hide)
-    )
-    (property "Datasheet" "http://www.ti.com/lit/gpn/sn74LS04" (id 3) (at -3.81 189.23 0)
-      (effects (font (size 1.27 1.27)) hide)
-    )
-  )
   (symbol (lib_id "74xx:74LS04") (at 55.88 110.49 0) (unit 2)
     (in_bom yes) (on_board yes)
@@
     )
   )
+  (symbol (lib_id "74xx:74LS04") (at 95.25 179.07 90) (unit 6)
+    (in_bom yes) (on_board yes)
+    (property "Reference" "U8" (id 0) (at 87.1982 179.07 0))
+    (property "Value" "74LS04" (id 1) (at 89.5096 179.07 0))
+    (property "Footprint" "" (id 2) (at 95.25 179.07 0)
+      (effects (font (size 1.27 1.27)) hide)
+    )
+    (property "Datasheet" "http://www.ti.com/lit/gpn/sn74LS04" (id 3) (at 95.25 179.07 0)
+      (effects (font (size 1.27 1.27)) hide)
+    )
+  )
   (symbol (lib_id "74xx:74LS04") (at 213.36 133.35 270) (unit 1)
     (in_bom yes) (on_board yes)
@@
     )
   )
-  (symbol (lib_id "74xx:74LS01") (at 34.29 231.14 0) (mirror y) (unit 1)
-    (in_bom yes) (on_board yes)
-    (property "Reference" "U4" (id 0) (at 34.29 222.885 0))
-    (property "Value" "74LS01" (id 1) (at 34.29 225.1964 0))
-    (property "Footprint" "" (id 2) (at 34.29 231.14 0)
-      (effects (font (size 1.27 1.27)) hide)
-    )
-    (property "Datasheet" "http://www.nteinc.com/specs/7400to7499/pdf/nte74LS01.pdf" (id 3) (at 34.29 231.14 0)
+  (symbol (lib_id "74xx:74LS01") (at 34.29 208.28 0) (mirror y) (unit 1)
+    (in_bom yes) (on_board yes)
+    (property "Reference" "U4" (id 0) (at 34.29 200.025 0))
+    (property "Value" "74LS01" (id 1) (at 34.29 202.3364 0))
+    (property "Footprint" "" (id 2) (at 34.29 208.28 0)
+      (effects (font (size 1.27 1.27)) hide)
+    )
+    (property "Datasheet" "http://www.nteinc.com/specs/7400to7499/pdf/nte74LS01.pdf" (id 3) (at 34.29 208.28 0)
       (effects (font (size 1.27 1.27)) hide)
     )
@@
     )
   )
-  (symbol (lib_id "74xx:74LS74") (at 64.77 193.04 0) (unit 2)
-    (in_bom yes) (on_board yes)
-    (property "Reference" "U11" (id 0) (at 64.77 180.8226 0))
-    (property "Value" "74ALS74" (id 1) (at 64.77 183.134 0))
-    (property "Footprint" "" (id 2) (at 64.77 193.04 0)
-      (effects (font (size 1.27 1.27)) hide)
-    )
-    (property "Datasheet" "74xx/74hc_hct74.pdf" (id 3) (at 64.77 193.04 0)
-      (effects (font (size 1.27 1.27)) hide)
-    )
+  (symbol (lib_id "74xx:74LS74") (at 64.77 182.88 0) (unit 2)
+    (in_bom yes) (on_board yes)
+    (property "Reference" "U11" (id 0) (at 64.77 170.6626 0))
+    (property "Value" "74ALS74" (id 1) (at 64.77 172.974 0))
+    (property "Footprint" "" (id 2) (at 64.77 182.88 0)
+      (effects (font (size 1.27 1.27)) hide)
+    )
+    (property "Datasheet" "74xx/74hc_hct74.pdf" (id 3) (at 64.77 182.88 0)
+      (effects (font (size 1.27 1.27)) hide)
+    )

Commit message: a
Parts:
- added C?: 27pF, symbol Device:C
- added L?: 220uH, symbol Device:L
- added R?: 2.2k, symbol Device:R
Connections:
- net GND: now also C?.2
- net VCC: now also R?.1
- net at J1.36 (Pin_36), U2.1 (~G1), U3.1 (~G1): now also U10.5, U10.6
- net at U4.5: now also U11.10 (~S), U4.6, U5.10 (~S), R?.2
- net IR: now reaches U4.13
- net IR: now also J?.10 (Pin_10)
- net at U8.9: now also U8.10
- net at U8.11: now also L?.2
- net RESET: now reaches J?.12 (Pin_12)
- net RESET: now also C?.1, L?.1
- net A0 renamed A1
- no-connect marks 13 -> 18
Other:
- moved on the sheet: J1, U11A, U3, U4B, U4C, U4D, U5A, U5B, U8C, U8D, U8E, U8F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

Commit message: a
Connections:
- net GND: now also U11.2 (D), U7.8 (GND)
- net VCC: now also U1.20 (VCC), U7.16 (VCC), U?.14 (VCC)
- net at U4.2: now also U8.13
- net at U4.3: now also U4.11, U5.9 (Q)
- net at U4.12: now also U8.12
- no-connect marks 18 -> 20
Other:
- moved on the sheet: U4D, U8F
Changed lines of the file:
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@@
   (junction (at 50.8 82.55) (diameter 0.9144) (color 0 0 0 0))
   (junction (at 53.34 80.01) (diameter 0.9144) (color 0 0 0 0))
+  (junction (at 53.34 210.82) (diameter 0.9144) (color 0 0 0 0))
   (junction (at 55.88 77.47) (diameter 0.9144) (color 0 0 0 0))
   (junction (at 58.42 74.93) (diameter 0.9144) (color 0 0 0 0))
@@
   (no_connect (at 68.58 142.24))
   (no_connect (at 140.97 182.88))
+  (no_connect (at 171.45 158.75))
+  (no_connect (at 217.17 175.26))
   (no_connect (at 294.64 101.6))
   (no_connect (at 394.97 218.44))
@@
     (stroke (width 0) (type solid) (color 0 0 0 0))
   )
-  (wire (pts (xy 24.13 157.48) (xy 40.64 157.48))
+  (wire (pts (xy 24.13 157.48) (xy 30.48 157.48))
     (stroke (width 0) (type solid) (color 0 0 0 0))
   )
@@
     (stroke (width 0) (type solid) (color 0 0 0 0))
   )
+  (wire (pts (xy 41.91 205.74) (xy 49.53 205.74))
+    (stroke (width 0) (type solid) (color 0 0 0 0))
+  )
   (wire (pts (xy 45.72 100.33) (xy 2.54 100.33))
     (stroke (width 0) (type solid) (color 0 0 0 0))
@@
     (stroke (width 0) (type solid) (color 0 0 0 0))
   )
+  (wire (pts (xy 45.72 154.94) (xy 53.34 154.94))
+    (stroke (width 0) (type solid) (color 0 0 0 0))
+  )
   (wire (pts (xy 48.26 38.1) (xy 115.57 38.1))
     (stroke (width 0) (type solid) (color 0 0 0 0))
@@
     (stroke (width 0) (type solid) (color 0 0 0 0))
   )
+  (wire (pts (xy 49.53 160.02) (xy 45.72 160.02))
+    (stroke (width 0) (type solid) (color 0 0 0 0))
+  )
+  (wire (pts (xy 49.53 165.1) (xy 49.53 160.02))
+    (stroke (width 0) (type solid) (color 0 0 0 0))
+  )
+  (wire (pts (xy 49.53 205.74) (xy 49.53 180.34))
+    (stroke (width 0) (type solid) (color 0 0 0 0))
+  )
   (wire (pts (xy 50.8 40.64) (xy 118.11 40.64))
     (stroke (width 0) (type solid) (color 0 0 0 0))
@@
     (stroke (width 0) (type solid) (color 0 0 0 0))
   )
+  (wire (pts (xy 53.34 154.94) (xy 53.34 210.82))
+    (stroke (width 0) (type solid) (color 0 0 0 0))
+  )
+  (wire (pts (xy 53.34 210.82) (xy 41.91 210.82))
+    (stroke (width 0) (type solid) (color 0 0 0 0))
+  )
   (wire (pts (xy 55.88 45.72) (xy 123.19 45.72))
     (stroke (width 0) (type solid) (color 0 0 0 0))
@@
     (stroke (width 0) (type solid) (color 0 0 0 0))
   )
+  (wire (pts (xy 87.63 180.34) (xy 93.98 180.34))
+    (stroke (width 0) (type solid) (color 0 0 0 0))
+  )
+  (wire (pts (xy 87.63 191.77) (xy 87.63 180.34))
+    (stroke (width 0) (type solid) (color 0 0 0 0))
+  )
   (wire (pts (xy 93.98 67.31) (xy 96.52 67.31))
     (stroke (width 0) (type solid) (color 0 0 0 0))
@@
   )
   (wire (pts (xy 207.01 173.99) (xy 125.73 173.99))
+    (stroke (width 0) (type solid) (color 0 0 0 0))
+  )
+  (wire (pts (xy 212.09 175.26) (xy 212.09 210.82))
+    (stroke (width 0) (type solid) (color 0 0 0 0))
+  )
+  (wire (pts (xy 212.09 210.82) (xy 53.34 210.82))
     (stroke (width 0) (type solid) (color 0 0 0 0))
   )
@@
     )
   )
+  (symbol (lib_id "power:VCC") (at 81.28 59.69 0) (unit 1)
+    (in_bom yes) (on_board yes)
+    (property "Reference" "#PWR?" (id 0) (at 81.28 63.5 0)
+      (effects (font (size 1.27 1.27)) hide)
+    )
+    (property "Value" "VCC" (id 1) (at 82.55 54.61 0))
+    (property "Footprint" "" (id 2) (at 81.28 59.69 0)
+      (effects (font (size 1.27 1.27)) hide)
+    )
+    (property "Datasheet" "" (id 3) (at 81.28 59.69 0)
+      (effects (font (size 1.27 1.27)) hide)
+    )
+  )
+  (symbol (lib_id "power:VCC") (at 81.28 116.84 0) (unit 1)
+    (in_bom yes) (on_board yes)
+    (property "Reference" "#PWR?" (id 0) (at 81.28 120.65 0)
+      (effects (font (size 1.27 1.27)) hide)
+    )
+    (property "Value" "VCC" (id 1) (at 82.55 111.76 0))
+    (property "Footprint" "" (id 2) (at 81.28 116.84 0)
+      (effects (font (size 1.27 1.27)) hide)
+    )
+    (property "Datasheet" "" (id 3) (at 81.28 116.84 0)
+      (effects (font (size 1.27 1.27)) hide)
+    )
+  )
   (symbol (lib_id "power:VCC") (at 233.68 234.95 0) (unit 1)
     (in_bom yes) (on_board yes)
@@
     )
     (property "Datasheet" "" (id 3) (at 233.68 234.95 0)
+      (effects (font (size 1.27 1.27)) hide)
+    )
+  )
+  (symbol (lib_id "power:VCC") (at 281.94 93.98 0) (unit 1)
+    (in_bom yes) (on_board yes)
+    (property "Reference" "#PWR?" (id 0) (at 281.94 97.79 0)
+      (effects (font (size 1.27 1.27)) hide)
+    )
+    (property "Value" "VCC" (id 1) (at 283.21 88.9 0))
+    (property "Footprint" "" (id 2) (at 281.94 93.98 0)
+      (effects (font (size 1.27 1.27)) hide)
+    )
+    (property "Datasheet" "" (id 3) (at 281.94 93.98 0)
       (effects (font (size 1.27 1.27)) hide)
     )
@@
     )
   )
+  (symbol (lib_id "power:GND") (at 81.28 152.4 0) (unit 1)
+    (in_bom yes) (on_board yes)
+    (property "Reference" "#PWR?" (id 0) (at 81.28 158.75 0)
+      (effects (font (size 1.27 1.27)) hide)
+    )
+    (property "Value" "GND" (id 1) (at 82.55 157.48 0))
+    (property "Footprint" "" (id 2) (at 81.28 152.4 0)
+      (effects (font (size 1.27 1.27)) hide)
+    )
+    (property "Datasheet" "" (id 3) (at 81.28 152.4 0)
+      (effects (font (size 1.27 1.27)) hide)
+    )
+  )
+  (symbol (lib_id "power:GND") (at 87.63 191.77 0) (unit 1)
+    (in_bom yes) (on_board yes)
+    (property "Reference" "#PWR?" (id 0) (at 87.63 198.12 0)
+      (effects (font (size 1.27 1.27)) hide)
+    )
+    (property "Value" "GND" (id 1) (at 88.9 196.85 0))
+    (property "Footprint" "" (id 2) (at 87.63 191.77 0)
+      (effects (font (size 1.27 1.27)) hide)
+    )
+    (property "Datasheet" "" (id 3) (at 87.63 191.77 0)
+      (effects (font (size 1.27 1.27)) hide)
+    )
+  )
   (symbol (lib_id "power:GND") (at 119.38 147.32 0) (unit 1)
     (in_bom yes) (on_board yes)
@@
     )
   )
-  (symbol (lib_id "74xx:74LS04") (at 52.07 171.45 90) (unit 6)
-    (in_bom yes) (on_board yes)
-    (property "Reference" "U8" (id 0) (at 44.0182 171.45 0))
-    (property "Value" "74LS04" (id 1) (at 46.3296 171.45 0))
-    (property "Footprint" "" (id 2) (at 52.07 171.45 0)
-      (effects (font (size 1.27 1.27)) hide)
-    )
-    (property "Datasheet" "http://www.ti.com/lit/gpn/sn74LS04" (id 3) (at 52.07 171.45 0)
+  (symbol (lib_id "74xx:74LS04") (at 49.53 172.72 90) (unit 6)
+    (in_bom yes) (on_board yes)
+    (property "Reference" "U8" (id 0) (at 41.4782 172.72 0))
+    (property "Value" "74LS04" (id 1) (at 43.7896 172.72 0))
+    (property "Footprint" "" (id 2) (at 49.53 172.72 0)
+      (effects (font (size 1.27 1.27)) hide)
+    )
+    (property "Datasheet" "http://www.ti.com/lit/gpn/sn74LS04" (id 3) (at 49.53 172.72 0)
       (effects (font (size 1.27 1.27)) hide)
     )
@@
     )
   )
-  (symbol (lib_id "74xx:74LS01") (at 48.26 157.48 0) (mirror y) (unit 4)
-    (in_bom yes) (on_board yes)
-    (property "Reference" "U4" (id 0) (at 48.26 149.225 0))
-    (property "Value" "74LS01" (id 1) (at 48.26 151.5364 0))
-    (property "Footprint" "" (id 2) (at 48.26 157.48 0)
-      (effects (font (size 1.27 1.27)) hide)
-    )
-    (property "Datasheet" "http://www.nteinc.com/specs/7400to7499/pdf/nte74LS01.pdf" (id 3) (at 48.26 157.48 0)
+  (symbol (lib_id "74xx:74LS01") (at 38.1 157.48 0) (mirror y) (unit 4)
+    (in_bom yes) (on_board yes)
+    (property "Reference" "U4" (id 0) (at 38.1 149.225 0))
+    (property "Value" "74LS01" (id 1) (at 38.1 151.5364 0))
+    (property "Footprint" "" (id 2) (at 38.1 157.48 0)
+      (effects (font (size 1.27 1.27)) hide)
+    )
+    (property "Datasheet" "http://www.nteinc.com/specs/7400to7499/pdf/nte74LS01.pdf" (id 3) (at 38.1 157.48 0)
       (effects (font (size 1.27 1.27)) hide)
     )
@@
   )
   (symbol_instances
+    (path "/014534ad-89f1-451f-9531-635481df5d06"
+      (reference "#PWR?") (unit 1) (value "VCC") (footprint "")
+    )
     (path "/1d7f2762-8573-43bb-b630-29d449a1c414"
       (reference "#PWR?") (unit 1) (value "GND") (footprint "")
@@
       (reference "#PWR?") (unit 1) (value "GND") (footprint "")
     )
+    (path "/564ee8f0-170b-486c-bc39-5da2643cf3b7"
+      (reference "#PWR?") (unit 1) (value "GND") (footprint "")
+    )
     (path "/58b6dc4f-6436-4473-82fa-1b206df4d314"
       (reference "#PWR?") (unit 1) (value "GND") (footprint "")
@@
       (reference "#PWR?") (unit 1) (value "GND") (footprint "")
     )
+    (path "/92891b0a-c129-4534-8b44-116b13c280dc"
+      (reference "#PWR?") (unit 1) (value "VCC") (footprint "")
+    )
+    (path "/a0bc0353-f9d8-4833-9c6b-dbf743f46178"
+      (reference "#PWR?") (unit 1) (value "GND") (footprint "")
+    )
     (path "/a6363c87-506c-46a7-88f5-75efedfd6f5c"
       (reference "#PWR?") (unit 1) (value "VCC") (footprint "")
@@
       (reference "#PWR?") (unit 1) (value "VCC") (footprint "")
     )
+    (path "/df2eb90e-0203-44fe-8d90-67fdc0be7e52"
+      (reference "#PWR?") (unit 1) (value "VCC") (footprint "")
+    )
