File: acsi_to_scsi.kicad_sch (KiCad schematic)
At the start: 19 parts, among them J1 SCSI, U1 74ALS573, U10 74LS02, U11 74ALS74, U2 74ALS540, U3 74ALS540, U4 74LS01, U5 74ALS74, U6 74ALS08, U7 74ALS85, U8 74LS04, U9 74LS08

Commit message: a
Connections:
- net at U2.2 (A0): now also J1.2 (Pin_2), U3.18 (~B0), U?.8 (A)
- net at U2.3 (A1): now also J1.4 (Pin_4), U3.17 (~B1), U?.9 (B)
- net at U2.4 (A2): now also J1.6 (Pin_6), U3.16 (~B2), U?.10 (C)
- net at U2.5 (A3): now also J1.8 (Pin_8), U3.15 (~B3), U?.11 (D)
- net at U2.6 (A4): now also J1.10 (Pin_10), U3.14 (~B4), U?.12 (E)
- net at U2.7 (A5): now also J1.12 (Pin_12), U3.13 (~B5), U?.13 (F)
- net at U2.8 (A6): now also J1.14 (Pin_14), U3.12 (~B6), U?.1 (G)
- net at U2.9 (A7): now also J1.16 (Pin_16), U3.11 (~B7), U?.2 (H)
- net at U10.2: now also U10.4
