File: acsi_to_scsi.kicad_sch (KiCad schematic)
At the start: 19 parts, among them J1 SCSI, U1 74ALS573, U10 74LS02, U11 74ALS74, U2 74ALS540, U3 74ALS540, U4 74LS01, U5 74ALS74, U6 74ALS08, U7 74ALS85, U8 74LS04, U9 74LS08

Commit message: a
Connections:
- net GND: now also U5.2 (D)
- net at U1.12 (Q7), U7.11 (B1): now also U6.4
- net at U1.13 (Q6), U7.14 (B2): now also U6.12
- net at U1.14 (Q5), U7.1 (B3): now also U6.1
- net at U3.19 (~G2): now also U9.8
- net at U5.1 (~R): now also U5.12 (D), U6.8
- net at U5.3 (C): now also U8.2
- net at U5.4 (~S): now also U5.11 (C), U8.6
- net at U5.5 (Q): now also J1.38 (Pin_38)
- net at U5.13 (~R): now also U10.13
- net at U6.9: now also J1.48 (Pin_48), U8.5
Other:
- moved on the sheet: U10A, U10D, U8A

Commit message: a
Connections:
- net at U1.11 (Load), U9.11: now also U10.11, U8.1
- net at J1.2 (Pin_2), U2.2 (A0), U3.18 (~B0)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: now also U4.10
- net at U4.8: now also U11.9 (Q), U4.9
- net at U7.6 (Oa=b): now also U11.12 (D)
- net at U8.10, U8.9: now also U10.12, U10.3
- net at U10.1: now also U11.13 (~R)
- no-connect marks 20 -> 21
Other:
- moved on the sheet: U4C, U?

Commit message: a
Connections:
- net GND: now also U7.2 (Ia<b)
- net at U4.2, U8.13: now also J1.46 (Pin_46)
- net at U6.10, U6.13, U6.2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: now also U11.6 (~Q)
- net at J1.48 (Pin_48), U8.5: now also U11.3 (C); no longer U6.9
- net at J1.40 (Pin_40), U8.8: now also U11.1 (~R)
- net at U11.4 (~S): now also J1.44 (Pin_44), U11.8 (~Q)
- net at J1.42 (Pin_42): now also U6.9
- no-connect marks 21 -> 22
Changed lines of the file:
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@@
   (junction (at 26.67 139.7) (diameter 0.9144) (color 0 0 0 0))
   (junction (at 48.26 85.09) (diameter 0.9144) (color 0 0 0 0))
+  (junction (at 49.53 205.74) (diameter 0.9144) (color 0 0 0 0))
   (junction (at 50.8 82.55) (diameter 0.9144) (color 0 0 0 0))
   (junction (at 53.34 80.01) (diameter 0.9144) (color 0 0 0 0))
@@
   (junction (at 66.04 67.31) (diameter 0.9144) (color 0 0 0 0))
   (junction (at 81.28 100.33) (diameter 0.9144) (color 0 0 0 0))
+  (junction (at 83.82 208.28) (diameter 0.9144) (color 0 0 0 0))
+  (junction (at 97.79 132.08) (diameter 0.9144) (color 0 0 0 0))
   (junction (at 99.06 114.3) (diameter 0.9144) (color 0 0 0 0))
   (junction (at 101.6 121.92) (diameter 0.9144) (color 0 0 0 0))
@@
   (junction (at 138.43 127) (diameter 0.9144) (color 0 0 0 0))
   (junction (at 138.43 140.97) (diameter 0.9144) (color 0 0 0 0))
+  (junction (at 138.43 154.94) (diameter 0.9144) (color 0 0 0 0))
   (junction (at 165.1 58.42) (diameter 0.9144) (color 0 0 0 0))
   (junction (at 167.64 111.76) (diameter 0.9144) (color 0 0 0 0))
@@
   (junction (at 379.73 220.98) (diameter 0.9144) (color 0 0 0 0))
   (junction (at 393.7 125.73) (diameter 0.9144) (color 0 0 0 0))
+  (junction (at 396.24 115.57) (diameter 0.9144) (color 0 0 0 0))
   (junction (at 397.51 137.16) (diameter 0.9144) (color 0 0 0 0))
   (junction (at 400.05 205.74) (diameter 0.9144) (color 0 0 0 0))
@@
   (no_connect (at 400.05 100.33))
   (no_connect (at 400.05 102.87))
+  (no_connect (at 400.05 107.95))
   (no_connect (at 412.75 97.79))
   (no_connect (at 415.29 203.2))
@@
     (stroke (width 0) (type solid) (color 0 0 0 0))
   )
+  (wire (pts (xy 49.53 215.9) (xy 49.53 205.74))
+    (stroke (width 0) (type solid) (color 0 0 0 0))
+  )
   (wire (pts (xy 50.8 40.64) (xy 118.11 40.64))
     (stroke (width 0) (type solid) (color 0 0 0 0))
@@
     (stroke (width 0) (type solid) (color 0 0 0 0))
   )
+  (wire (pts (xy 66.04 118.11) (xy 97.79 118.11))
+    (stroke (width 0) (type solid) (color 0 0 0 0))
+  )
+  (wire (pts (xy 66.04 127) (xy 66.04 118.11))
+    (stroke (width 0) (type solid) (color 0 0 0 0))
+  )
   (wire (pts (xy 68.58 100.33) (xy 68.58 92.71))
     (stroke (width 0) (type solid) (color 0 0 0 0))
   )
+  (wire (pts (xy 68.58 127) (xy 66.04 127))
+    (stroke (width 0) (type solid) (color 0 0 0 0))
+  )
   (wire (pts (xy 68.58 129.54) (xy 64.77 129.54))
     (stroke (width 0) (type solid) (color 0 0 0 0))
   )
+  (wire (pts (xy 72.39 185.42) (xy 72.39 208.28))
+    (stroke (width 0) (type solid) (color 0 0 0 0))
+  )
+  (wire (pts (xy 72.39 208.28) (xy 83.82 208.28))
+    (stroke (width 0) (type solid) (color 0 0 0 0))
+  )
   (wire (pts (xy 80.01 180.34) (xy 72.39 180.34))
     (stroke (width 0) (type solid) (color 0 0 0 0))
@@
     (stroke (width 0) (type solid) (color 0 0 0 0))
   )
+  (wire (pts (xy 83.82 175.26) (xy 83.82 208.28))
+    (stroke (width 0) (type solid) (color 0 0 0 0))
+  )
+  (wire (pts (xy 83.82 208.28) (xy 370.84 208.28))
+    (stroke (width 0) (type solid) (color 0 0 0 0))
+  )
   (wire (pts (xy 87.63 180.34) (xy 93.98 180.34))
     (stroke (width 0) (type solid) (color 0 0 0 0))
@@
     (stroke (width 0) (type solid) (color 0 0 0 0))
   )
-  (wire (pts (xy 93.98 132.08) (xy 119.38 132.08))
+  (wire (pts (xy 93.98 132.08) (xy 97.79 132.08))
     (stroke (width 0) (type solid) (color 0 0 0 0))
   )
@@
     (stroke (width 0) (type solid) (color 0 0 0 0))
   )
+  (wire (pts (xy 93.98 198.12) (xy 93.98 182.88))
+    (stroke (width 0) (type solid) (color 0 0 0 0))
+  )
   (wire (pts (xy 96.52 67.31) (xy 96.52 22.86))
     (stroke (width 0) (type solid) (color 0 0 0 0))
@@
     (stroke (width 0) (type solid) (color 0 0 0 0))
   )
+  (wire (pts (xy 97.79 118.11) (xy 97.79 132.08))
+    (stroke (width 0) (type solid) (color 0 0 0 0))
+  )
+  (wire (pts (xy 97.79 132.08) (xy 119.38 132.08))
+    (stroke (width 0) (type solid) (color 0 0 0 0))
+  )
   (wire (pts (xy 99.06 20.32) (xy 204.47 20.32))
     (stroke (width 0) (type solid) (color 0 0 0 0))
@@
     (stroke (width 0) (type solid) (color 0 0 0 0))
   )
+  (wire (pts (xy 101.6 175.26) (xy 83.82 175.26))
+    (stroke (width 0) (type solid) (color 0 0 0 0))
+  )
+  (wire (pts (xy 101.6 196.85) (xy 101.6 190.5))
+    (stroke (width 0) (type solid) (color 0 0 0 0))
+  )
   (wire (pts (xy 104.14 15.24) (xy 104.14 74.93))
     (stroke (width 0) (type solid) (color 0 0 0 0))
@@
     (stroke (width 0) (type solid) (color 0 0 0 0))
   )
+  (wire (pts (xy 109.22 185.42) (xy 120.65 185.42))
+    (stroke (width 0) (type solid) (color 0 0 0 0))
+  )
   (wire (pts (xy 115.57 38.1) (xy 115.57 85.09))
     (stroke (width 0) (type solid) (color 0 0 0 0))
@@
     (stroke (width 0) (type solid) (color 0 0 0 0))
   )
+  (wire (pts (xy 120.65 154.94) (xy 138.43 154.94))
+    (stroke (width 0) (type solid) (color 0 0 0 0))
+  )
+  (wire (pts (xy 120.65 185.42) (xy 120.65 154.94))
+    (stroke (width 0) (type solid) (color 0 0 0 0))
+  )
   (wire (pts (xy 123.19 45.72) (xy 123.19 77.47))
     (stroke (width 0) (type solid) (color 0 0 0 0))
@@
     (stroke (width 0) (type solid) (color 0 0 0 0))
   )
+  (wire (pts (xy 345.44 123.19) (xy 345.44 215.9))
+    (stroke (width 0) (type solid) (color 0 0 0 0))
+  )
+  (wire (pts (xy 345.44 215.9) (xy 49.53 215.9))
+    (stroke (width 0) (type solid) (color 0 0 0 0))
+  )
   (wire (pts (xy 363.22 115.57) (xy 367.03 115.57))
     (stroke (width 0) (type solid) (color 0 0 0 0))
@@
     (stroke (width 0) (type solid) (color 0 0 0 0))
   )
+  (wire (pts (xy 368.3 118.11) (xy 368.3 133.35))
+    (stroke (width 0) (type solid) (color 0 0 0 0))
+  )
+  (wire (pts (xy 368.3 133.35) (xy 299.72 133.35))
+    (stroke (width 0) (type solid) (color 0 0 0 0))
+  )
+  (wire (pts (xy 370.84 120.65) (xy 400.05 120.65))
+    (stroke (width 0) (type solid) (color 0 0 0 0))
+  )
+  (wire (pts (xy 370.84 208.28) (xy 370.84 120.65))
+    (stroke (width 0) (type solid) (color 0 0 0 0))
+  )
   (wire (pts (xy 374.65 125.73) (xy 374.65 152.4))
     (stroke (width 0) (type solid) (color 0 0 0 0))
   )
+  (wire (pts (xy 378.46 134.62) (xy 378.46 198.12))
+    (stroke (width 0) (type solid) (color 0 0 0 0))
+  )
+  (wire (pts (xy 378.46 198.12) (xy 93.98 198.12))
+    (stroke (width 0) (type solid) (color 0 0 0 0))
+  )
   (wire (pts (xy 379.73 215.9) (xy 379.73 220.98))
     (stroke (width 0) (type solid) (color 0 0 0 0))
@@
     (stroke (width 0) (type solid) (color 0 0 0 0))
   )
-  (wire (pts (xy 393.7 125.73) (xy 393.7 133.35))
+  (wire (pts (xy 393.7 125.73) (xy 393.7 134.62))
     (stroke (width 0) (type solid) (color 0 0 0 0))
   )
@@
     (stroke (width 0) (type solid) (color 0 0 0 0))
   )
-  (wire (pts (xy 393.7 133.35) (xy 299.72 133.35))
+  (wire (pts (xy 393.7 134.62) (xy 378.46 134.62))
+    (stroke (width 0) (type solid) (color 0 0 0 0))
+  )
+  (wire (pts (xy 396.24 115.57) (xy 388.62 115.57))
+    (stroke (width 0) (type solid) (color 0 0 0 0))
+  )
+  (wire (pts (xy 396.24 115.57) (xy 396.24 196.85))
+    (stroke (width 0) (type solid) (color 0 0 0 0))
+  )
+  (wire (pts (xy 396.24 196.85) (xy 101.6 196.85))
     (stroke (width 0) (type solid) (color 0 0 0 0))
   )
@@
     (stroke (width 0) (type solid) (color 0 0 0 0))
   )
-  (wire (pts (xy 400.05 115.57) (xy 388.62 115.57))
-    (stroke (width 0) (type solid) (color 0 0 0 0))
-  )
+  (wire (pts (xy 400.05 115.57) (xy 396.24 115.57))
+    (stroke (width 0) (type solid) (color 0 0 0 0))
+  )
+  (wire (pts (xy 400.05 118.11) (xy 368.3 118.11))
+    (stroke (width 0) (type solid) (color 0 0 0 0))
+  )
+  (wire (pts (xy 400.05 123.19) (xy 345.44 123.19))
+    (stroke (width 0) (type solid) (color 0 0 0 0))
+  )

Commit message: a
Parts:
- gave numbers to parts that had none: 7
Connections:
- net at J1.36 (Pin_36), U10.5, U10.6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: now also J1.2 (Pin_2), U12.8 (A), U2.2 (A0), U3.18 (~B0), U4.10
- net at U3.19 (~G2), U9.8: now also J1.48 (Pin_48), U11.3 (C), U8.5
Other:
- moved on the sheet: J1, J2, R1, SW1, U1, U10A, U10B, U10C, U10D, U10E, U11A, U11B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

Commit message: a
Parts:
- C1: footprint (none) -> Capacitor_THT:C_Disc_D3.0mm_W1.6mm_P2.50mm
- J1: footprint (none) -> Connector_PinHeader_2.54mm:PinHeader_2x25_P2.54mm_Horizontal
- J2: footprint (none) -> Connector_PinHeader_2.54mm:PinHeader_1x19_P2.54mm_Horizontal
- L1: footprint (none) -> Inductor_THT:L_Axial_L5.0mm_D3.6mm_P10.00mm_Horizontal_Murata_BL01RN1A2A2
- R1, R2: footprint (none) -> Resistor_THT:R_Axial_DIN0204_L3.6mm_D1.6mm_P1.90mm_Vertical
- SW1: footprint (none) -> Button_Switch_THT:SW_DIP_SPSTx03_Slide_9.78x9.8mm_W7.62mm_P2.54mm
- U1, U2, U3: footprint (none) -> Package_DIP:DIP-20_W7.62mm
- U10, U11, U12, U4, U5, U6, U8, U9: footprint (none) -> Package_DIP:DIP-14_W7.62mm
- U7: footprint (none) -> Package_DIP:DIP-16_W7.62mm

Commit message: a
Parts:
- removed U4: 74LS01, Package_DIP:DIP-14_W7.62mm, symbol 74xx:74LS01
- added U4: 74LS00, symbol 74xx:74LS00
Connections:
- net DR: now also U4.3
- net GND: now also U4.7 (GND)
- net IR: now also U4.11
- net VCC: now also U4.14 (VCC)
- net at J1.2 (Pin_2), J1.36 (Pin_36), U10.5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: now also U4.8
- net at J1.46 (Pin_46), U8.13: now also U4.2
- net at U5.9 (Q): now also U4.1, U4.13
- net at R1.2, U11.10 (~S), U5.10 (~S): now also U4.4, U4.5
- net at U11.9 (Q): now also U4.10, U4.9
- net at U8.12: now also U4.12
Changed lines of the file:
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@@
     (stroke (width 0) (type solid) (color 0 0 0 0))
   )
-  (wire (pts (xy 144.78 185.42) (xy 144.78 180.34))
+  (wire (pts (xy 144.78 180.34) (xy 144.78 185.42))
     (stroke (width 0) (type solid) (color 0 0 0 0))
   )
@@
     (stroke (width 0) (type solid) (color 0 0 0 0))
   )
+  (wire (pts (xy 156.21 251.46) (xy 180.34 251.46))
+    (stroke (width 0) (type solid) (color 0 0 0 0))
+  )
   (wire (pts (xy 157.48 106.68) (xy 157.48 127))
     (stroke (width 0) (type solid) (color 0 0 0 0))
@@
   )
   (wire (pts (xy 180.34 226.06) (xy 199.39 226.06))
-    (stroke (width 0) (type solid) (color 0 0 0 0))
-  )
-  (wire (pts (xy 180.34 251.46) (xy 156.21 251.46))
     (stroke (width 0) (type solid) (color 0 0 0 0))
   )
@@
     )
   )
-  (symbol (lib_id "74xx:74LS01") (at 53.34 208.28 0) (mirror y) (unit 1)
-    (in_bom yes) (on_board yes)
-    (property "Reference" "U4" (id 0) (at 53.34 200.025 0))
-    (property "Value" "74LS01" (id 1) (at 53.34 202.3364 0))
-    (property "Footprint" "Package_DIP:DIP-14_W7.62mm" (id 2) (at 53.34 208.28 0)
-      (effects (font (size 1.27 1.27)) hide)
-    )
-    (property "Datasheet" "http://www.nteinc.com/specs/7400to7499/pdf/nte74LS01.pdf" (id 3) (at 53.34 208.28 0)
+  (symbol (lib_id "74xx:74LS00") (at 53.34 208.28 180) (unit 1)
+    (in_bom yes) (on_board yes)
+    (property "Reference" "U4" (id 0) (at 53.34 199.39 0))
+    (property "Value" "74LS00" (id 1) (at 53.34 201.93 0))
+    (property "Footprint" "" (id 2) (at 53.34 208.28 0)
+      (effects (font (size 1.27 1.27)) hide)
+    )
+    (property "Datasheet" "http://www.ti.com/lit/gpn/sn74ls00" (id 3) (at 53.34 208.28 0)
       (effects (font (size 1.27 1.27)) hide)
     )
@@
     )
   )
-  (symbol (lib_id "74xx:74LS01") (at 57.15 157.48 0) (mirror y) (unit 4)
-    (in_bom yes) (on_board yes)
-    (property "Reference" "U4" (id 0) (at 57.15 149.225 0))
-    (property "Value" "74LS01" (id 1) (at 57.15 151.5364 0))
-    (property "Footprint" "Package_DIP:DIP-14_W7.62mm" (id 2) (at 57.15 157.48 0)
-      (effects (font (size 1.27 1.27)) hide)
-    )
-    (property "Datasheet" "http://www.nteinc.com/specs/7400to7499/pdf/nte74LS01.pdf" (id 3) (at 57.15 157.48 0)
+  (symbol (lib_id "74xx:74LS00") (at 57.15 157.48 180) (unit 4)
+    (in_bom yes) (on_board yes)
+    (property "Reference" "U4" (id 0) (at 57.15 148.59 0))
+    (property "Value" "74LS00" (id 1) (at 57.15 151.13 0))
+    (property "Footprint" "" (id 2) (at 57.15 157.48 0)
+      (effects (font (size 1.27 1.27)) hide)
+    )
+    (property "Datasheet" "http://www.ti.com/lit/gpn/sn74ls00" (id 3) (at 57.15 157.48 0)
       (effects (font (size 1.27 1.27)) hide)
     )
@@
     )
   )
-  (symbol (lib_id "74xx:74LS01") (at 152.4 182.88 0) (unit 2)
-    (in_bom yes) (on_board yes)
-    (property "Reference" "U4" (id 0) (at 152.4 174.625 0))
-    (property "Value" "74LS01" (id 1) (at 152.4 176.9364 0))
-    (property "Footprint" "Package_DIP:DIP-14_W7.62mm" (id 2) (at 152.4 182.88 0)
-      (effects (font (size 1.27 1.27)) hide)
-    )
-    (property "Datasheet" "http://www.nteinc.com/specs/7400to7499/pdf/nte74LS01.pdf" (id 3) (at 152.4 182.88 0)
+  (symbol (lib_id "74xx:74LS00") (at 152.4 182.88 0) (unit 2)
+    (in_bom yes) (on_board yes)
+    (property "Reference" "U4" (id 0) (at 152.4 173.99 0))
+    (property "Value" "74LS00" (id 1) (at 152.4 176.53 0))
+    (property "Footprint" "" (id 2) (at 152.4 182.88 0)
+      (effects (font (size 1.27 1.27)) hide)
+    )
+    (property "Datasheet" "http://www.ti.com/lit/gpn/sn74ls00" (id 3) (at 152.4 182.88 0)
       (effects (font (size 1.27 1.27)) hide)
     )
@@
     )
   )
-  (symbol (lib_id "74xx:74LS01") (at 200.66 191.77 0) (unit 3)
-    (in_bom yes) (on_board yes)
-    (property "Reference" "U4" (id 0) (at 200.66 183.515 0))
-    (property "Value" "74LS01" (id 1) (at 200.66 185.8264 0))
-    (property "Footprint" "Package_DIP:DIP-14_W7.62mm" (id 2) (at 200.66 191.77 0)
-      (effects (font (size 1.27 1.27)) hide)
-    )
-    (property "Datasheet" "http://www.nteinc.com/specs/7400to7499/pdf/nte74LS01.pdf" (id 3) (at 200.66 191.77 0)
+  (symbol (lib_id "74xx:74LS00") (at 200.66 191.77 0) (unit 3)
+    (in_bom yes) (on_board yes)
+    (property "Reference" "U4" (id 0) (at 200.66 182.88 0))
+    (property "Value" "74LS00" (id 1) (at 200.66 185.42 0))
+    (property "Footprint" "" (id 2) (at 200.66 191.77 0)
+      (effects (font (size 1.27 1.27)) hide)
+    )
+    (property "Datasheet" "http://www.ti.com/lit/gpn/sn74ls00" (id 3) (at 200.66 191.77 0)
       (effects (font (size 1.27 1.27)) hide)
     )
@@
     )
   )
-  (symbol (lib_id "74xx:74LS01") (at 180.34 238.76 0) (unit 5)
-    (in_bom yes) (on_board yes)
-    (property "Reference" "U4" (id 0) (at 186.182 237.5916 0)
-      (effects (font (size 1.27 1.27)) (justify left))
-    )
-    (property "Value" "74LS01" (id 1) (at 186.182 239.903 0)
-      (effects (font (size 1.27 1.27)) (justify left))
-    )
-    (property "Footprint" "Package_DIP:DIP-14_W7.62mm" (id 2) (at 180.34 238.76 0)
-      (effects (font (size 1.27 1.27)) hide)
-    )
-    (property "Datasheet" "http://www.nteinc.com/specs/7400to7499/pdf/nte74LS01.pdf" (id 3) (at 180.34 238.76 0)
+  (symbol (lib_id "74xx:74LS00") (at 180.34 238.76 0) (unit 5)
+    (in_bom yes) (on_board yes)
+    (property "Reference" "U4" (id 0) (at 186.69 237.49 0)
+      (effects (font (size 1.27 1.27)) (justify left))
+    )
+    (property "Value" "74LS00" (id 1) (at 186.69 240.03 0)
+      (effects (font (size 1.27 1.27)) (justify left))
+    )
+    (property "Footprint" "" (id 2) (at 180.34 238.76 0)
+      (effects (font (size 1.27 1.27)) hide)
+    )
+    (property "Datasheet" "http://www.ti.com/lit/gpn/sn74ls00" (id 3) (at 180.34 238.76 0)
       (effects (font (size 1.27 1.27)) hide)
     )
@@
       (reference "U3") (unit 1) (value "74ALS540") (footprint "Package_DIP:DIP-20_W7.62mm")
     )
-    (path "/00000000-0000-0000-0000-00005fc462a5"
-      (reference "U4") (unit 1) (value "74LS01") (footprint "Package_DIP:DIP-14_W7.62mm")
-    )
-    (path "/00000000-0000-0000-0000-00005fc47a03"
-      (reference "U4") (unit 2) (value "74LS01") (footprint "Package_DIP:DIP-14_W7.62mm")
-    )
-    (path "/00000000-0000-0000-0000-00005fc47dea"
-      (reference "U4") (unit 3) (value "74LS01") (footprint "Package_DIP:DIP-14_W7.62mm")
-    )
-    (path "/00000000-0000-0000-0000-00005fc481cc"
-      (reference "U4") (unit 4) (value "74LS01") (footprint "Package_DIP:DIP-14_W7.62mm")
-    )
-    (path "/00000000-0000-0000-0000-00005fc4862e"
-      (reference "U4") (unit 5) (value "74LS01") (footprint "Package_DIP:DIP-14_W7.62mm")
+    (path "/21267300-479e-4479-aa80-92bc66a06e40"
+      (reference "U4") (unit 1) (value "74LS00") (footprint "")
+    )
+    (path "/ac5659b7-d4a1-494d-8952-0a7749d41e47"
+      (reference "U4") (unit 2) (value "74LS00") (footprint "")
+    )
+    (path "/65225cb6-b8d0-41b2-a765-a872e2376741"
+      (reference "U4") (unit 3) (value "74LS00") (footprint "")
+    )
+    (path "/b281da9b-d1ed-4cb1-b491-f6ff3b8c8c72"
+      (reference "U4") (unit 4) (value "74LS00") (footprint "")
+    )
+    (path "/1d664e93-7bf8-4ea9-9d3d-58fb801f9324"
+      (reference "U4") (unit 5) (value "74LS00") (footprint "")
     )
     (path "/00000000-0000-0000-0000-00005fc4998d"

Commit message: init
Parts:
- U1: footprint Package_DIP:DIP-20_W7.62mm -> Package_SO:SOIC-20W_7.5x12.8mm_P1.27mm; DigiKey (none) -> 296-1129-1-ND
- U10: value 74LS02 -> 74ALS02; footprint Package_DIP:DIP-14_W7.62mm -> Package_SO:SOIC-14_3.9x8.7mm_P1.27mm; DigiKey (none) -> 296-5002-5-ND
- U11, U5: footprint Package_DIP:DIP-14_W7.62mm -> Package_SO:SO-14_5.3x10.2mm_P1.27mm; DigiKey (none) -> 296-53302-ND
- U12: footprint Package_DIP:DIP-14_W7.62mm -> Package_SO:SOIC-14_3.9x8.7mm_P1.27mm; DigiKey (none) -> SN74LS280D-ND
- U2, U3: footprint Package_DIP:DIP-20_W7.62mm -> Package_SO:SO-20_5.3x12.6mm_P1.27mm; DigiKey (none) -> 296-53300-ND
- U4: value 74LS00 -> 74ALS00; footprint (none) -> Package_SO:SOIC-14_3.9x8.7mm_P1.27mm; DigiKey (none) -> 296-1477-5-ND
- U6: footprint Package_DIP:DIP-14_W7.62mm -> Package_SO:SO-14_5.3x10.2mm_P1.27mm; DigiKey (none) -> 296-53296-ND
- U7: value 74ALS85 -> 74LS85; footprint Package_DIP:DIP-16_W7.62mm -> Package_SO:SOIC-16_3.9x9.9mm_P1.27mm; DigiKey (none) -> 296-49902-1-ND
- U8: value 74LS04 -> 74ALS04; footprint Package_DIP:DIP-14_W7.62mm -> Package_SO:SO-14_5.3x10.2mm_P1.27mm; DigiKey (none) -> 296-53295-ND
- U9: value 74LS08 -> 74ALS08; footprint Package_DIP:DIP-14_W7.62mm -> Package_SO:SO-14_5.3x10.2mm_P1.27mm; DigiKey (none) -> 296-53296-ND
