File: acsi_to_scsi.kicad_pcb (KiCad board)
At the start: 2 copper layers, 305 x 175 mm, 0 parts

Commit message: a
Parts:
- added C1: 27pF, Capacitor_THT:C_Disc_D3.0mm_W1.6mm_P2.50mm, F.Cu at (199.0, 165.0)
- added J1: SCSI, Connector_PinHeader_2.54mm:PinHeader_2x25_P2.54mm_Horizontal, F.Cu at (170.4, 119.3)
- added J2: ACSI, Connector_PinHeader_2.54mm:PinHeader_1x19_P2.54mm_Horizontal, F.Cu at (186.3, 119.3)
- added L1: 220uH, Inductor_THT:L_Axial_L5.0mm_D3.6mm_P10.00mm_Horizontal_Murata_BL01RN1A2A2, F.Cu at (169.7, 185.2)
- added R1: 2.2k, Resistor_THT:R_Axial_DIN0204_L3.6mm_D1.6mm_P1.90mm_Vertical, F.Cu at (169.7, 189.3)
- added R2: 1k, Resistor_THT:R_Axial_DIN0204_L3.6mm_D1.6mm_P1.90mm_Vertical, F.Cu at (174.6, 189.3)
- added SW1: SW_DIP_x03, Button_Switch_THT:SW_DIP_SPSTx03_Slide_9.78x9.8mm_W7.62mm_P2.54mm, F.Cu at (207.7, 166.7)
- added U1: 74ALS573, Package_DIP:DIP-20_W7.62mm, F.Cu at (220.8, 119.1)
- added U10: 74LS02, Package_DIP:DIP-14_W7.62mm, F.Cu at (199.1, 146.1)
- added U11: 74ALS74, Package_DIP:DIP-14_W7.62mm, F.Cu at (209.9, 146.1)
- added U12: 74LS280, Package_DIP:DIP-14_W7.62mm, F.Cu at (185.7, 169.4)
- added U2: 74ALS540, Package_DIP:DIP-20_W7.62mm, F.Cu at (199.1, 119.1)
- added U3: 74ALS540, Package_DIP:DIP-20_W7.62mm, F.Cu at (209.9, 119.1)
- added U4: 74LS01, Package_DIP:DIP-14_W7.62mm, F.Cu at (253.3, 119.1)
- added U5: 74ALS74, Package_DIP:DIP-14_W7.62mm, F.Cu at (231.6, 141.0)
- added U6: 74ALS08, Package_DIP:DIP-14_W7.62mm, F.Cu at (242.4, 119.1)
- added U7: 74ALS85, Package_DIP:DIP-16_W7.62mm, F.Cu at (231.6, 119.1)
- added U8: 74LS04, Package_DIP:DIP-14_W7.62mm, F.Cu at (196.5, 169.4)
- added U9: 74LS08, Package_DIP:DIP-14_W7.62mm, F.Cu at (220.8, 146.1)

Commit message: a
Parts:
- J2: footprint Connector_PinHeader_2.54mm:PinHeader_1x19_P2.54mm_Horizontal -> Connector_Dsub:DSUB-25_Female_Horizontal_P2.77x2.84mm_EdgePinOffset7.70mm_Housed_MountingHolesOffset9.12mm
- moved U7 138.6 mm to (94.0, 135.3), turned to 90 degrees
- moved U9 138.3 mm to (82.5, 150.5), turned to 90 degrees
- moved SW1 133.7 mm to (79.4, 128.9)
- moved U4 132.3 mm to (123.8, 92.1), turned to 90 degrees
- moved U3 119.6 mm to (90.8, 108.6), turned to 90 degrees
- moved C1 117.7 mm to (126.4, 72.4)
- moved L1 117.1 mm to (134.0, 73.7)
- moved U2 111.6 mm to (90.8, 92.1), turned to 90 degrees
- moved J2 105.9 mm to (95.2, 65.4), turned to 180 degrees
- moved U6 103.1 mm to (139.7, 127.0), turned to -90 degrees
- moved U1 101.3 mm to (120.0, 108.6), turned to 90 degrees
- moved U5 90.2 mm to (152.4, 97.8), turned to 90 degrees
- moved U8 81.3 mm to (131.4, 120.7), turned to 90 degrees
- moved R1 71.4 mm to (155.6, 119.4)
- moved R2 64.8 mm to (117.5, 158.8), turned to 180 degrees
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
Commit message: a
Parts:
- moved U6 16.2 mm to (125.7, 135.3), turned to 90 degrees
Changed lines of the file:
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@@
   )
   (footprint "Package_DIP:DIP-14_W7.62mm" (layer "F.Cu")
-    (at 139.7 127 -90)
+    (at 125.73 135.255 90)
     (descr "14-lead though-hole mounted DIP package, row spacing 7.62 mm (300 mils)")
     (tags "THT DIP DIL PDIP 2.54mm 7.62mm 300mil")
@@
     (fp_line (start 6.985 16.51) (end 0.635 16.51) (layer "F.Fab") (width 0.1))
     (fp_line (start 0.635 16.51) (end 0.635 -0.27) (layer "F.Fab") (width 0.1))
-    (pad "1" thru_hole rect (at 0 0 270) (locked) (size 1.6 1.6) (drill 0.8) (layers *.Cu *.Mask)
+    (pad "1" thru_hole rect (at 0 0 90) (locked) (size 1.6 1.6) (drill 0.8) (layers *.Cu *.Mask)
       (net 56 "Net-(U1-Pad14)"))
-    (pad "2" thru_hole oval (at 0 2.54 270) (locked) (size 1.6 1.6) (drill 0.8) (layers *.Cu *.Mask)
+    (pad "2" thru_hole oval (at 0 2.54 90) (locked) (size 1.6 1.6) (drill 0.8) (layers *.Cu *.Mask)
       (net 74 "Net-(U11-Pad6)"))
-    (pad "3" thru_hole oval (at 0 5.08 270) (locked) (size 1.6 1.6) (drill 0.8) (layers *.Cu *.Mask)
+    (pad "3" thru_hole oval (at 0 5.08 90) (locked) (size 1.6 1.6) (drill 0.8) (layers *.Cu *.Mask)
       (net 63 "Net-(U3-Pad7)"))
-    (pad "4" thru_hole oval (at 0 7.62 270) (locked) (size 1.6 1.6) (drill 0.8) (layers *.Cu *.Mask)
+    (pad "4" thru_hole oval (at 0 7.62 90) (locked) (size 1.6 1.6) (drill 0.8) (layers *.Cu *.Mask)
       (net 58 "Net-(U1-Pad12)"))
-    (pad "5" thru_hole oval (at 0 10.16 270) (locked) (size 1.6 1.6) (drill 0.8) (layers *.Cu *.Mask)
+    (pad "5" thru_hole oval (at 0 10.16 90) (locked) (size 1.6 1.6) (drill 0.8) (layers *.Cu *.Mask)
       (net 74 "Net-(U11-Pad6)"))
-    (pad "6" thru_hole oval (at 0 12.7 270) (locked) (size 1.6 1.6) (drill 0.8) (layers *.Cu *.Mask)
+    (pad "6" thru_hole oval (at 0 12.7 90) (locked) (size 1.6 1.6) (drill 0.8) (layers *.Cu *.Mask)
       (net 61 "Net-(U3-Pad9)"))
-    (pad "7" thru_hole oval (at 0 15.24 270) (locked) (size 1.6 1.6) (drill 0.8) (layers *.Cu *.Mask)
+    (pad "7" thru_hole oval (at 0 15.24 90) (locked) (size 1.6 1.6) (drill 0.8) (layers *.Cu *.Mask)
       (net 1 "GND") (pinfunction "GND"))
-    (pad "8" thru_hole oval (at 7.62 15.24 270) (locked) (size 1.6 1.6) (drill 0.8) (layers *.Cu *.Mask)
+    (pad "8" thru_hole oval (at 7.62 15.24 90) (locked) (size 1.6 1.6) (drill 0.8) (layers *.Cu *.Mask)
       (net 70 "Net-(U5-Pad1)"))
-    (pad "9" thru_hole oval (at 7.62 12.7 270) (locked) (size 1.6 1.6) (drill 0.8) (layers *.Cu *.Mask)
+    (pad "9" thru_hole oval (at 7.62 12.7 90) (locked) (size 1.6 1.6) (drill 0.8) (layers *.Cu *.Mask)
       (net 7 "Net-(U6-Pad9)"))
-    (pad "10" thru_hole oval (at 7.62 10.16 270) (locked) (size 1.6 1.6) (drill 0.8) (layers *.Cu *.Mask)
+    (pad "10" thru_hole oval (at 7.62 10.16 90) (locked) (size 1.6 1.6) (drill 0.8) (layers *.Cu *.Mask)
       (net 74 "Net-(U11-Pad6)"))
-    (pad "11" thru_hole oval (at 7.62 7.62 270) (locked) (size 1.6 1.6) (drill 0.8) (layers *.Cu *.Mask)
+    (pad "11" thru_hole oval (at 7.62 7.62 90) (locked) (size 1.6 1.6) (drill 0.8) (layers *.Cu *.Mask)
       (net 62 "Net-(U3-Pad8)"))
-    (pad "12" thru_hole oval (at 7.62 5.08 270) (locked) (size 1.6 1.6) (drill 0.8) (layers *.Cu *.Mask)
+    (pad "12" thru_hole oval (at 7.62 5.08 90) (locked) (size 1.6 1.6) (drill 0.8) (layers *.Cu *.Mask)
       (net 57 "Net-(U1-Pad13)"))
-    (pad "13" thru_hole oval (at 7.62 2.54 270) (locked) (size 1.6 1.6) (drill 0.8) (layers *.Cu *.Mask)
+    (pad "13" thru_hole oval (at 7.62 2.54 90) (locked) (size 1.6 1.6) (drill 0.8) (layers *.Cu *.Mask)
       (net 74 "Net-(U11-Pad6)"))
-    (pad "14" thru_hole oval (at 7.62 0 270) (locked) (size 1.6 1.6) (drill 0.8) (layers *.Cu *.Mask)
+    (pad "14" thru_hole oval (at 7.62 0 90) (locked) (size 1.6 1.6) (drill 0.8) (layers *.Cu *.Mask)
       (net 15 "VCC") (pinfunction "VCC"))
     (model "${KICAD6_3DMODEL_DIR}/Package_DIP.3dshapes/DIP-14_W7.62mm.wrl"
