File: _autosave-acsi_to_scsi.kicad_pcb (KiCad board)
At the start: 2 copper layers, 305 x 175 mm, 20 parts, among them J1 SCSI, J2 ACSI, SW1 SW_DIP_x03, U1 74ALS573, U10 74ALS02, U11 74ALS74, U12 74LS280, U2 74ALS540, U3 74ALS540, U4 74ALS00, U4 74LS01, U5 74ALS74, U6 74ALS08, U7 74LS85, U8 74ALS04, U9 74ALS08

Commit message: init
Parts:
- removed the U4 at (123.8, 92.1)
- moved U2 36.9 mm to (106.6, 125.5)
- moved U3 14.8 mm to (85.0, 95.0)
